File: KiCad/Sw_Mat_RGB_R.kicad_sch (KiCad schematic)
At the start: 200 parts, among them SW108 MACRO4, SW37 F7, SW38 F8, SW39 F9, SW40 F10, SW41 11, SW42 F12, SW43 PRT_SCR, SW44 DEL, SW45 7, SW46 8, SW47 9, SW48 0, SW49 -, SW50 =, SW51 BACKSPACE, SW52 R_SPACE, SW53 Y, SW54 U, SW55 I, SW56 O, SW57 P, SW58 [, SW59 ], SW60 R_ALT, SW61 H, SW62 J, SW63 K, SW64 L, SW65 ;, SW66 ', SW67 ENTER, SW68 FN, SW69 N, SW70 M, SW71 ,, SW72 ., SW73 /, SW74 R_SHIFT, SW75 UP, SW76 R_CTRL, SW77 LEFT, SW78 DOWN, SW79 \, SW80 RIGHT, SW81 MACRO1, SW82 MACRO2, SW83 MACRO3

Commit message: Updated Readme and switch matrix
Parts:
- SW41: value 11 -> F11
Changed lines of the file:
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@@
     (in_bom yes) (on_board yes)
     (property "Reference" "SW41" (id 0) (at 295.91 64.77 0))
-    (property "Value" "11" (id 1) (at 295.91 66.675 0))
+    (property "Value" "F11" (id 1) (at 295.91 66.675 0))
     (property "Footprint" "Button_Switch_Keyboard:SW_Cherry_MX_1.00u_PCB" (id 2) (at 295.91 70.485 0)
       (effects (font (size 1.27 1.27)) hide)
