File: Esquemáticos y PCB/mechpad/SWITCH_MATRIX_RGB_LEFT.kicad_sch (KiCad schematic)
At the start: 151 parts, among them SW1 ESC, SW10 3, SW11 4, SW12 5, SW13 TAB, SW14 Q, SW15 W, SW16 E, SW17 R, SW18 T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

Commit message: Updated schematic
Added connections between hierarchical sheets, more code testing
Parts:
- gave numbers to parts that had none: 7
- renumbered C3 to C10, C4 to C11, C5 to C12, C6 to C13, C7 to C14, C8 to C15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
