File: Esquemáticos y PCB/mechpad/SWITCH_MATRIX_RGB_RIGHT.kicad_sch (KiCad schematic)
At the start: 209 parts, among them SW108 MACRO4, SW37 F7, SW38 F8, SW39 F9, SW40 F10, SW41 F11, SW42 F12, SW43 PRT_SCR, SW44 DEL, SW45 7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

Commit message: Updated schematic
Added connections between hierarchical sheets, more code testing
Parts:
- renumbered C37 to C44, C38 to C45, C39 to C46, C40 to C47, C41 to C48, C42 to C49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
