File: Schematics and PCB/Li-Po_Charge_Boost.kicad_sch (KiCad schematic)
At the start: 29 parts, among them Q1 FS8205, SW107 Battery Switch, U19 TLV71311PDBVR, U20 TLV70033DDCR, U7 TP4056, U8 MT3608, U9 FS312F-G

Commit message: Right layout created
Parts:
- removed C211, C212, C213, C214: 1u X5R, symbol Device:C
- removed U19: TLV71311PDBVR, Package_TO_SOT_SMD:TSOT-23-5, symbol Regulator_Linear:ADP7182AUJZ-1.8
- removed U20: TLV70033DDCR, Package_TO_SOT_SMD:TSOT-23-5, symbol Regulator_Linear:ADP7182AUJZ-1.8
Other:
- note removed: "Lower Voltage LDOs"
