File: Schematics and PCB/Li-Po_Charge_Boost.kicad_sch (KiCad schematic)
At the start: 23 parts, among them Q1 FS8205, SW107 Battery Switch, U7 TP4056, U8 MT3608, U9 FS312F-G

Commit message: Finished initial iteration of the Right layout
Parts:
- renumbered R111 to R109
Changed lines of the file:
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@@
       (project "Schematics and PCB"
         (path "/e4b186e2-256b-418b-b9a4-327a6681c2f1/0f61d57d-7083-4e3b-b040-dc8971ea63c8"
-          (reference "R112") (unit 1)
+          (reference "R110") (unit 1)
         )
       )
@@
       (project "Schematics and PCB"
         (path "/e4b186e2-256b-418b-b9a4-327a6681c2f1/0f61d57d-7083-4e3b-b040-dc8971ea63c8"
-          (reference "R109") (unit 1)
+          (reference "R107") (unit 1)
         )
       )
@@
       (project "Schematics and PCB"
         (path "/e4b186e2-256b-418b-b9a4-327a6681c2f1/0f61d57d-7083-4e3b-b040-dc8971ea63c8"
-          (reference "#PWR0436") (unit 1)
+          (reference "#PWR0542") (unit 1)
         )
       )
@@
       (project "Schematics and PCB"
         (path "/e4b186e2-256b-418b-b9a4-327a6681c2f1/0f61d57d-7083-4e3b-b040-dc8971ea63c8"
-          (reference "R106") (unit 1)
+          (reference "R104") (unit 1)
         )
       )
@@
       (project "Schematics and PCB"
         (path "/e4b186e2-256b-418b-b9a4-327a6681c2f1/0f61d57d-7083-4e3b-b040-dc8971ea63c8"
-          (reference "R110") (unit 1)
+          (reference "R108") (unit 1)
         )
       )
@@
       (project "Schematics and PCB"
         (path "/e4b186e2-256b-418b-b9a4-327a6681c2f1/0f61d57d-7083-4e3b-b040-dc8971ea63c8"
-          (reference "#PWR0432") (unit 1)
+          (reference "#PWR0540") (unit 1)
         )
       )
@@
       (project "Schematics and PCB"
         (path "/e4b186e2-256b-418b-b9a4-327a6681c2f1/0f61d57d-7083-4e3b-b040-dc8971ea63c8"
-          (reference "U24") (unit 1)
+          (reference "U23") (unit 1)
         )
       )
@@
       (project "Schematics and PCB"
         (path "/e4b186e2-256b-418b-b9a4-327a6681c2f1/0f61d57d-7083-4e3b-b040-dc8971ea63c8"
-          (reference "R107") (unit 1)
+          (reference "R105") (unit 1)
         )
       )
@@
       (project "Schematics and PCB"
         (path "/e4b186e2-256b-418b-b9a4-327a6681c2f1/0f61d57d-7083-4e3b-b040-dc8971ea63c8"
-          (reference "#PWR0431") (unit 1)
+          (reference "#PWR0539") (unit 1)
         )
       )
@@
       (project "Schematics and PCB"
         (path "/e4b186e2-256b-418b-b9a4-327a6681c2f1/0f61d57d-7083-4e3b-b040-dc8971ea63c8"
-          (reference "#PWR0440") (unit 1)
+          (reference "#PWR0545") (unit 1)
         )
       )
@@
       (project "Schematics and PCB"
         (path "/e4b186e2-256b-418b-b9a4-327a6681c2f1/0f61d57d-7083-4e3b-b040-dc8971ea63c8"
-          (reference "C211") (unit 1)
+          (reference "C213") (unit 1)
         )
       )
@@
       (project "Schematics and PCB"
         (path "/e4b186e2-256b-418b-b9a4-327a6681c2f1/0f61d57d-7083-4e3b-b040-dc8971ea63c8"
-          (reference "R105") (unit 1)
+          (reference "R103") (unit 1)
         )
       )
@@
       (project "Schematics and PCB"
         (path "/e4b186e2-256b-418b-b9a4-327a6681c2f1/0f61d57d-7083-4e3b-b040-dc8971ea63c8"
-          (reference "C207") (unit 1)
+          (reference "C211") (unit 1)
         )
       )
@@
       (project "Schematics and PCB"
         (path "/e4b186e2-256b-418b-b9a4-327a6681c2f1/0f61d57d-7083-4e3b-b040-dc8971ea63c8"
-          (reference "#PWR0438") (unit 1)
+          (reference "#PWR0543") (unit 1)
         )
       )
@@
       (project "Schematics and PCB"
         (path "/e4b186e2-256b-418b-b9a4-327a6681c2f1/0f61d57d-7083-4e3b-b040-dc8971ea63c8"
-          (reference "R108") (unit 1)
+          (reference "R106") (unit 1)
         )
       )
@@
   (symbol (lib_id "Device:R_US") (at 149.225 87.63 90) (unit 1)
     (in_bom yes) (on_board yes) (dnp no)
-    (property "Reference" "R111" (at 149.225 90.17 90)
+    (property "Reference" "R109" (at 149.225 90.17 90)
       (effects (font (size 1.27 1.27)))
     )
@@
       (project "Schematics and PCB"
         (path "/e4b186e2-256b-418b-b9a4-327a6681c2f1/0f61d57d-7083-4e3b-b040-dc8971ea63c8"
-          (reference "R111") (unit 1)
+          (reference "R109") (unit 1)
         )
       )
@@
       (project "Schematics and PCB"
         (path "/e4b186e2-256b-418b-b9a4-327a6681c2f1/0f61d57d-7083-4e3b-b040-dc8971ea63c8"
-          (reference "U20") (unit 1)
+          (reference "U21") (unit 1)
         )
       )
@@
       (project "Schematics and PCB"
         (path "/e4b186e2-256b-418b-b9a4-327a6681c2f1/0f61d57d-7083-4e3b-b040-dc8971ea63c8"
-          (reference "#PWR0437") (unit 1)
+          (reference "#PWR0541") (unit 1)
         )
       )
@@
       (project "Schematics and PCB"
         (path "/e4b186e2-256b-418b-b9a4-327a6681c2f1/0f61d57d-7083-4e3b-b040-dc8971ea63c8"
-          (reference "D130") (unit 1)
+          (reference "D129") (unit 1)
         )
       )
@@
       (project "Schematics and PCB"
         (path "/e4b186e2-256b-418b-b9a4-327a6681c2f1/0f61d57d-7083-4e3b-b040-dc8971ea63c8"
-          (reference "D128") (unit 1)
+          (reference "D127") (unit 1)
         )
       )
@@
       (project "Schematics and PCB"
         (path "/e4b186e2-256b-418b-b9a4-327a6681c2f1/0f61d57d-7083-4e3b-b040-dc8971ea63c8"
-          (reference "#PWR0441") (unit 1)
+          (reference "#PWR0546") (unit 1)
         )
       )
@@
       (project "Schematics and PCB"
         (path "/e4b186e2-256b-418b-b9a4-327a6681c2f1/0f61d57d-7083-4e3b-b040-dc8971ea63c8"
-          (reference "#PWR0446") (unit 1)
+          (reference "#PWR0548") (unit 1)
         )
       )
@@
       (project "Schematics and PCB"
         (path "/e4b186e2-256b-418b-b9a4-327a6681c2f1/0f61d57d-7083-4e3b-b040-dc8971ea63c8"
-          (reference "R113") (unit 1)
+          (reference "R111") (unit 1)
         )
       )
@@
       (project "Schematics and PCB"
         (path "/e4b186e2-256b-418b-b9a4-327a6681c2f1/0f61d57d-7083-4e3b-b040-dc8971ea63c8"
-          (reference "C210") (unit 1)
+          (reference "C212") (unit 1)
         )
       )
@@
       (project "Schematics and PCB"
         (path "/e4b186e2-256b-418b-b9a4-327a6681c2f1/0f61d57d-7083-4e3b-b040-dc8971ea63c8"
-          (reference "#PWR0445") (unit 1)
+          (reference "#PWR0547") (unit 1)
         )
       )
@@
       (project "Schematics and PCB"
         (path "/e4b186e2-256b-418b-b9a4-327a6681c2f1/0f61d57d-7083-4e3b-b040-dc8971ea63c8"
-          (reference "D129") (unit 1)
+          (reference "D128") (unit 1)
         )
       )
@@
       (project "Schematics and PCB"
         (path "/e4b186e2-256b-418b-b9a4-327a6681c2f1/0f61d57d-7083-4e3b-b040-dc8971ea63c8"
-          (reference "#PWR0439") (unit 1)
-        )
-      )
+          (reference "#PWR0544") (unit 1)
+        )
+      )
