File: Schematics and PCB/shiftRegister.kicad_sch (KiCad schematic)
At the start: 1 part, among them U1 74HC165

Commit message: Right layout created
Parts:
- removed U1: 74HC165, symbol 74xx:74HC165
Connections:
- no-connect marks 2 -> 0
Changed lines of the file:
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@@
 (kicad_sch (version 20230121) (generator eeschema)
   (paper "A4")
-  (no_connect (at 116.84 77.47))
-  (no_connect (at 91.44 77.47))
-  (hierarchical_label "GND" (shape input) (at 104.14 118.11 270) (fields_autoplaced)
-    (effects (font (size 1.27 1.27)) (justify right))
-  )
-  (hierarchical_label "D5" (shape input) (at 91.44 92.71 180) (fields_autoplaced)
-    (effects (font (size 1.27 1.27)) (justify right))
-  )
-  (hierarchical_label "D0" (shape input) (at 91.44 80.01 180) (fields_autoplaced)
-    (effects (font (size 1.27 1.27)) (justify right))
-  )
-  (hierarchical_label "D4" (shape input) (at 91.44 90.17 180) (fields_autoplaced)
-    (effects (font (size 1.27 1.27)) (justify right))
-  )
-  (hierarchical_label "D3" (shape input) (at 91.44 87.63 180) (fields_autoplaced)
-    (effects (font (size 1.27 1.27)) (justify right))
-  )
-  (hierarchical_label "D7" (shape input) (at 91.44 97.79 180) (fields_autoplaced)
-    (effects (font (size 1.27 1.27)) (justify right))
-  )
-  (hierarchical_label "~{PL}" (shape input) (at 91.44 102.87 180) (fields_autoplaced)
-    (effects (font (size 1.27 1.27)) (justify right))
-  )
-  (hierarchical_label "~{Q}" (shape input) (at 116.84 80.01 0) (fields_autoplaced)
-    (effects (font (size 1.27 1.27)) (justify left))
-  )
-  (hierarchical_label "+5V" (shape input) (at 104.14 69.85 90) (fields_autoplaced)
-    (effects (font (size 1.27 1.27)) (justify left))
-  )
-  (hierarchical_label "D1" (shape input) (at 91.44 82.55 180) (fields_autoplaced)
-    (effects (font (size 1.27 1.27)) (justify right))
-  )
-  (hierarchical_label "D2" (shape input) (at 91.44 85.09 180) (fields_autoplaced)
-    (effects (font (size 1.27 1.27)) (justify right))
-  )
-  (hierarchical_label "D6" (shape input) (at 91.44 95.25 180) (fields_autoplaced)
-    (effects (font (size 1.27 1.27)) (justify right))
-  )
-  (hierarchical_label "~{CE}" (shape input) (at 91.44 110.49 180) (fields_autoplaced)
-    (effects (font (size 1.27 1.27)) (justify right))
-  )
-  (hierarchical_label "CP" (shape input) (at 91.44 107.95 180) (fields_autoplaced)
-    (effects (font (size 1.27 1.27)) (justify right))
-  )
-  (symbol (lib_id "74xx:74HC165") (at 104.14 92.71 0) (unit 1)
-    (in_bom yes) (on_board yes) (dnp no) (fields_autoplaced)
-    (property "Reference" "U1" (at 106.4093 71.12 0)
-      (effects (font (size 1.27 1.27)) (justify left))
-    )
-    (property "Value" "74HC165" (at 106.4093 73.66 0)
-      (effects (font (size 1.27 1.27)) (justify left))
-    )
-    (property "Footprint" "" (at 104.14 92.71 0)
-      (effects (font (size 1.27 1.27)) hide)
-    )
-    (property "Datasheet" "https://assets.nexperia.com/documents/data-sheet/74HC_HCT165.pdf" (at 104.14 92.71 0)
-      (effects (font (size 1.27 1.27)) hide)
-    )
-    (pin "1")
-    (pin "10")
-    (pin "11")
-    (pin "12")
-    (pin "13")
-    (pin "14")
-    (pin "15")
-    (pin "16")
-    (pin "2")
-    (pin "3")
-    (pin "4")
-    (pin "5")
-    (pin "6")
-    (pin "7")
-    (pin "8")
-    (pin "9")
-    (instances
-      (project "mechpad"
-        (path "/2d068e7d-d024-48f7-a9a1-e9ed75f7807b"
-          (reference "U1") (unit 1)
-        )
-        (path "/2d068e7d-d024-48f7-a9a1-e9ed75f7807b/85c1e75e-627d-4c70-b3a6-c94424fb96f2"
-          (reference "U3") (unit 1)
-        )
-      )
-      (project "Schematics and PCB"
-        (path "/e4b186e2-256b-418b-b9a4-327a6681c2f1"
-          (reference "U5") (unit 1)
-        )
-        (path "/e4b186e2-256b-418b-b9a4-327a6681c2f1/80716739-d01c-4b0b-872b-3c2eebf89dc4"
-          (reference "U6") (unit 1)
-        )
-        (path "/e4b186e2-256b-418b-b9a4-327a6681c2f1/a273b463-3673-4820-9332-fbf118fc465f"
-          (reference "U15") (unit 1)
-        )
-        (path "/e4b186e2-256b-418b-b9a4-327a6681c2f1/c38bb0a6-c0de-42d5-8b44-d8a8437996f0"
-          (reference "U16") (unit 1)
-        )
-      )
-    )
-  )
 )
