File: Schematics and PCB/switchMatrixRight.kicad_sch (KiCad schematic)
At the start: 207 parts, among them SW37 F7, SW38 F8, SW39 F9, SW40 F10, SW41 F11, SW42 F12, SW43 PRT_SCR, SW44 DEL, SW45 7, SW46 8, SW47 9, SW48 0, SW49 -, SW50 =, SW51 BACKSPACE, SW52 MACRO1, SW53 Y, SW54 U, SW55 I, SW56 O, SW57 P, SW58 [, SW59 ], SW60 \, SW61 MACRO2, SW62 H, SW63 J, SW64 K, SW65 L, SW66 ;, SW67 ', SW68 ENTER, SW69 MACRO3, SW70 N, SW71 M, SW72 ,, SW73 ., SW74 /, SW75 R_SHIFT, SW76 UP, SW77 MACRO4, SW78 R_SPACE, SW79 R_ALT, SW80 FN, SW81 R_CTRL, SW82 LEFT, SW83 DOWN, SW84 RIGHT

Commit message: Right layout created
Parts:
- removed D48: 1N4148W, Diode_SMD:D_SOD-123, symbol Device:D
- removed R15: 10K, Resistor_SMD:R_0805_2012Metric, symbol Device:R_US
- added R28: 10k, symbol Device:R_US
- added U15: 74HC165, symbol mechpadLibrary:74HC165
- added U6: ~, symbol mechpadLibrary:74HC595
Connections:
- net RE_SW2 is gone; now on net GND: RE1.S2
- net +5V: now also R28.1, U15.16 (VCC), U6.10 (~{CLR}), U6.16 (VCC)
- net COL_0_R: now also SW78.1 (A), U15.11 (D0)
- net COL_1_R: now also SW79.1 (A), U15.12 (D1); no longer SW78.1 (A)
- net COL_2_R: now also SW80.1 (A), U15.13 (D2); no longer SW79.1 (A)
- net COL_3_R: now also SW81.1 (A), U15.14 (D3); no longer SW80.1 (A)
- net COL_4_R: now also SW82.1 (A), U15.3 (D4); no longer SW81.1 (A)
- net COL_5_R: now also SW83.1 (A), U15.4 (D5); no longer SW82.1 (A)
- net COL_6_R: now also SW84.1 (A), U15.5 (D6); no longer SW83.1 (A)
- net COL_7_R: now also SW52.1 (A), U15.6 (D7); no longer SW84.1 (A)
- net GND: now also U15.8 (GND), U6.13 (~{OE}), U6.8 (GND)
- net ROW_0_R: now also U6.15 (QA)
- net ROW_1_R: now also U6.1 (QB)
- net ROW_2_R: now also U6.2 (QC); no longer D65.1 (K)
- net ROW_3_R: now also D65.1 (K), U6.3 (QD); no longer D73.1 (K)
- net ROW_4_R: now also D73.1 (K), U6.4 (QE); no longer D81.1 (K)
- net ROW_5_R: now also D81.1 (K), U6.5 (QF)
- removed net COL_8_R: RE1.S1, SW52.1 (A), SW61.1 (A), SW69.1 (A), SW77.1 (A)
- new net CP: U15.2 (CP)
- new net DS: U6.14 (DS)
- new net RE_SW: R28.2, RE1.S1
- new net SH_CP: U6.11 (SH_CP)
- new net ST_CP: U6.12 (ST_CP)
- new net ~{CE}: U15.15 (~{CE})
- new net ~{PL}: U15.1 (~{PL})
- new net ~{Q7}: U15.7 (~{Q7})
- no-connect marks 0 -> 5
Other:
- moved on the sheet: C80, C81, D82, D83, D84, D85, D86, D87, D88, R24, R25, RE1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
