File: Schematics and PCB/switchMatrixRight.kicad_sch (KiCad schematic)
At the start: 209 parts, among them SW37 F7, SW38 F8, SW39 F9, SW40 F10, SW41 F11, SW42 F12, SW43 PRT_SCR, SW44 DEL, SW45 7, SW46 8, SW47 9, SW48 0, SW49 -, SW50 =, SW51 BACKSPACE, SW52 MACRO1, SW53 Y, SW54 U, SW55 I, SW56 O, SW57 P, SW58 [, SW59 ], SW60 \, SW61 MACRO2, SW62 H, SW63 J, SW64 K, SW65 L, SW66 ;, SW67 ', SW68 ENTER, SW69 MACRO3, SW70 N, SW71 M, SW72 ,, SW73 ., SW74 /, SW75 R_SHIFT, SW76 UP, SW77 MACRO4, SW78 R_SPACE, SW79 R_ALT, SW80 FN, SW81 R_CTRL, SW82 LEFT, SW83 DOWN, SW84 RIGHT

Commit message: Updated USB hub
Parts:
- C80, C81: value 10nF -> 10n

Commit message: Pre initial PCB layout commit
Parts:
- removed C44, C45, C46, C47, C48, C49, C50, C51, C52, C53, C54, C55, C56, C57, C58, C59, C60, C61, C62, C63, C64, C65, C66, C67, C68, C69, C70, C71, C72, C73, C74, C75, C76, C77, C78, C79, C82, C83, C84, C85, C86, C87, C88, C89, C90, C91, C92, C93: 100n, Capacitor_SMD:C_0603_1608Metric, symbol Device:C
- removed R16, R17, R18, R19, R20, R21, R22, R23, R26, R27: 10K, Resistor_SMD:R_0603_1608Metric, symbol Device:R_US
- removed RGB37, RGB38, RGB39, RGB40, RGB41, RGB42, RGB43, RGB44, RGB45, RGB46, RGB47, RGB48, RGB49, RGB50, RGB51, RGB52, RGB53, RGB54, RGB55, RGB56, RGB57, RGB58, RGB59, RGB60, RGB61, RGB62, RGB63, RGB64, RGB65, RGB66, RGB67, RGB68, RGB69, RGB70, RGB71, RGB72, RGB73, RGB74, RGB75, RGB76, RGB77, RGB78, RGB79, RGB80, RGB81, RGB82, RGB83, RGB84: WS2812B, LED_SMD:LED_WS2812B_PLCC4_5.0x5.0mm_P3.2mm, symbol LED:WS2812B
- added C44 (x48): 100n, Capacitor_SMD:C_0805_2012Metric, symbol Device:C
- added R15 (x8): 10K, Resistor_SMD:R_0805_2012Metric, symbol Device:R_US
- added RGB37 (x48): WS2812B, LED_SMD:LED_WS2812B_PLCC4_5.0x5.0mm_P3.2mm, symbol LED:WS2812B
- C80, C81: value 10n -> 100n
- R15: footprint Resistor_SMD:R_0603_1608Metric -> Resistor_SMD:R_0805_2012Metric
Connections:
- net +5V: now also C44.1, C44.1, C44.1, C44.1, C44.1, C44.1, C44.1, C44.1, C44.1, C44.1, C44.1, C44.1, C44.1, C44.1, C44.1, C44.1, C44.1, C44.1, C44.1, C44.1, C44.1, C44.1, C44.1, C44.1, C44.1, C44.1, C44.1, C44.1, C44.1, C44.1, C44.1, C44.1, C44.1, C44.1, C44.1, C44.1, C44.1, C44.1, C44.1, C44.1, C44.1, C44.1, C44.1, C44.1, C44.1, C44.1, C44.1, C44.1, R15.1, R15.1, R15.1, R15.1, R15.1, R15.1, R15.1, R15.1, RGB37.1 (VDD), RGB37.1 (VDD), RGB37.1 (VDD), RGB37.1 (VDD), RGB37.1 (VDD), RGB37.1 (VDD), RGB37.1 (VDD), RGB37.1 (VDD), RGB37.1 (VDD), RGB37.1 (VDD), RGB37.1 (VDD), RGB37.1 (VDD), RGB37.1 (VDD), RGB37.1 (VDD), RGB37.1 (VDD), RGB37.1 (VDD), RGB37.1 (VDD), RGB37.1 (VDD), RGB37.1 (VDD), RGB37.1 (VDD), RGB37.1 (VDD), RGB37.1 (VDD), RGB37.1 (VDD), RGB37.1 (VDD), RGB37.1 (VDD), RGB37.1 (VDD), RGB37.1 (VDD), RGB37.1 (VDD), RGB37.1 (VDD), RGB37.1 (VDD), RGB37.1 (VDD), RGB37.1 (VDD), RGB37.1 (VDD), RGB37.1 (VDD), RGB37.1 (VDD), RGB37.1 (VDD), RGB37.1 (VDD), RGB37.1 (VDD), RGB37.1 (VDD), RGB37.1 (VDD), RGB37.1 (VDD), RGB37.1 (VDD), RGB37.1 (VDD), RGB37.1 (VDD), RGB37.1 (VDD), RGB37.1 (VDD), RGB37.1 (VDD), RGB37.1 (VDD)
- net COL_1_R: now also R15.2
- net COL_2_R: now also R15.2
- net COL_3_R: now also R15.2
- net COL_4_R: now also R15.2
- net COL_5_R: now also R15.2
- net COL_6_R: now also R15.2
- net COL_7_R: now also R15.2
- net COL_8_R: now also R15.2
- net GND: now also C44.2, C44.2, C44.2, C44.2, C44.2, C44.2, C44.2, C44.2, C44.2, C44.2, C44.2, C44.2, C44.2, C44.2, C44.2, C44.2, C44.2, C44.2, C44.2, C44.2, C44.2, C44.2, C44.2, C44.2, C44.2, C44.2, C44.2, C44.2, C44.2, C44.2, C44.2, C44.2, C44.2, C44.2, C44.2, C44.2, C44.2, C44.2, C44.2, C44.2, C44.2, C44.2, C44.2, C44.2, C44.2, C44.2, C44.2, C44.2, RGB37.3 (VSS), RGB37.3 (VSS), RGB37.3 (VSS), RGB37.3 (VSS), RGB37.3 (VSS), RGB37.3 (VSS), RGB37.3 (VSS), RGB37.3 (VSS), RGB37.3 (VSS), RGB37.3 (VSS), RGB37.3 (VSS), RGB37.3 (VSS), RGB37.3 (VSS), RGB37.3 (VSS), RGB37.3 (VSS), RGB37.3 (VSS), RGB37.3 (VSS), RGB37.3 (VSS), RGB37.3 (VSS), RGB37.3 (VSS), RGB37.3 (VSS), RGB37.3 (VSS), RGB37.3 (VSS), RGB37.3 (VSS), RGB37.3 (VSS), RGB37.3 (VSS), RGB37.3 (VSS), RGB37.3 (VSS), RGB37.3 (VSS), RGB37.3 (VSS), RGB37.3 (VSS), RGB37.3 (VSS), RGB37.3 (VSS), RGB37.3 (VSS), RGB37.3 (VSS), RGB37.3 (VSS), RGB37.3 (VSS), RGB37.3 (VSS), RGB37.3 (VSS), RGB37.3 (VSS), RGB37.3 (VSS), RGB37.3 (VSS), RGB37.3 (VSS), RGB37.3 (VSS), RGB37.3 (VSS), RGB37.3 (VSS), RGB37.3 (VSS), RGB37.3 (VSS)
- net RE_1_A: now also R25.2, RE1.B
- net RE_1_B: now also R24.2, RE1.A
- net RGB_IN_R: now also RGB37.4 (DIN)
- net RGB_OUT_R: now also RGB37.2 (DOUT)
- new net: RGB37.2 (DOUT), RGB37.4 (DIN) (x47)
Other:
- moved on the sheet: C80, C81, D40, D41, D42, D43, D44, D45, D46, D47, D48, D49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

Commit message: minor changes
Parts:
- removed C44 (x47): 100n, Capacitor_SMD:C_0805_2012Metric, symbol Device:C
- removed R24, R25: 10K, Resistor_SMD:R_0603_1608Metric, symbol Device:R_US
- removed RGB37 (x47): WS2812B, LED_SMD:LED_WS2812B_PLCC4_5.0x5.0mm_P3.2mm, symbol LED:WS2812B
- added C100, C138, C139, C140, C141, C58, C59, C60, C61, C62, C63, C64, C65, C66, C67, C68, C69, C70, C71, C72, C73, C74, C75, C76, C77, C78, C79, C82, C83, C84, C85, C86, C87, C88, C89, C90, C91, C92, C93, C94, C95, C96, C97, C98, C99: 100n, Capacitor_SMD:C_0805_2012Metric, symbol Device:C
- added C135, C136, C137: 100n, Capacitor_SMD:C_0603_1608Metric, symbol Device:C
- added R55, R56: 10K, Resistor_SMD:R_0603_1608Metric, symbol Device:R_US
- added RGB106, RGB107, RGB108, RGB109, RGB110, RGB111, RGB112, RGB113, RGB114, RGB115, RGB116, RGB117, RGB118, RGB119, RGB120, RGB121, RGB122, RGB123, RGB124, RGB125, RGB126, RGB127, RGB128, RGB129, RGB130, RGB131, RGB132, RGB133, RGB134, RGB135, RGB136, RGB137, RGB138, RGB139, RGB140, RGB141, RGB142, RGB143, RGB144, RGB145, RGB146, RGB147, RGB148, RGB149, RGB150, RGB151, RGB152: WS2812B, LED_SMD:LED_WS2812B_PLCC4_5.0x5.0mm_P3.2mm, symbol LED:WS2812B
- C80, C81: footprint Capacitor_SMD:C_0603_1608Metric -> Capacitor_SMD:C_0805_2012Metric
- renumbered C44 to C57, D40 to D43, D41 to D44, D42 to D45, D43 to D46, D44 to D47, D45 to D48, D46 to D49, D47 to D50, D48 to D51, D49 to D52, D50 to D53, D51 to D54, D52 to D55, D53 to D56, D54 to D57, D55 to D58, D56 to D59, D57 to D60, D58 to D61, D59 to D62, D60 to D63, D61 to D64, D62 to D65, D63 to D66, D64 to D67, D65 to D68, D66 to D69, D67 to D70, D68 to D71, D69 to D72, D70 to D73, D71 to D74, D72 to D75, D73 to D76, D74 to D77, D75 to D78, D76 to D79, D77 to D80, D78 to D81, D79 to D82, D80 to D83, D81 to D84, D82 to D85, D83 to D86, D84 to D87, D85 to D88, D86 to D89, D87 to D90, D88 to D91, R15 to R20, R15 to R21, R15 to R22, R15 to R23, R15 to R24, R15 to R25, R15 to R26, R15 to R27, R15 to R28, RGB37 to RGB105, SW37 to SW38, SW38 to SW39, SW39 to SW40, SW40 to SW41, SW41 to SW42, SW42 to SW43, SW43 to SW44, SW44 to SW45, SW45 to SW46, SW46 to SW47, SW47 to SW48, SW48 to SW49, SW49 to SW50, SW50 to SW51, SW51 to SW52, SW52 to SW53, SW53 to SW54, SW54 to SW55, SW55 to SW56, SW56 to SW57, SW57 to SW58, SW58 to SW59, SW59 to SW60, SW60 to SW61, SW61 to SW62, SW62 to SW63, SW63 to SW64, SW64 to SW65, SW65 to SW66, SW66 to SW67, SW67 to SW68, SW68 to SW69, SW69 to SW70, SW70 to SW71, SW71 to SW72, SW72 to SW73, SW73 to SW74, SW74 to SW75, SW75 to SW76, SW76 to SW77, SW77 to SW78, SW78 to SW79, SW79 to SW80, SW80 to SW81, SW81 to SW82, SW82 to SW83, SW83 to SW84, SW84 to SW85
Connections:
- net +5V: now also C80.1, C81.1, C100.1, C138.1, C139.1, C140.1, C141.1, C58.1, C59.1, C60.1, C61.1, C62.1, C63.1, C64.1, C65.1, C66.1, C67.1, C68.1, C69.1, C70.1, C71.1, C72.1, C73.1, C74.1, C75.1, C76.1, C77.1, C78.1, C79.1, C82.1, C83.1, C84.1, C85.1, C86.1, C87.1, C88.1, C89.1, C90.1, C91.1, C92.1, C93.1, C94.1, C95.1, C96.1, C97.1, C98.1, C99.1, RGB106.1 (VDD), RGB107.1 (VDD), RGB108.1 (VDD), RGB109.1 (VDD), RGB110.1 (VDD), RGB111.1 (VDD), RGB112.1 (VDD), RGB113.1 (VDD), RGB114.1 (VDD), RGB115.1 (VDD), RGB116.1 (VDD), RGB117.1 (VDD), RGB118.1 (VDD), RGB119.1 (VDD), RGB120.1 (VDD), RGB121.1 (VDD), RGB122.1 (VDD), RGB123.1 (VDD), RGB124.1 (VDD), RGB125.1 (VDD), RGB126.1 (VDD), RGB127.1 (VDD), RGB128.1 (VDD), RGB129.1 (VDD), RGB130.1 (VDD), RGB131.1 (VDD), RGB132.1 (VDD), RGB133.1 (VDD), RGB134.1 (VDD), RGB135.1 (VDD), RGB136.1 (VDD), RGB137.1 (VDD), RGB138.1 (VDD), RGB139.1 (VDD), RGB140.1 (VDD), RGB141.1 (VDD), RGB142.1 (VDD), RGB143.1 (VDD), RGB144.1 (VDD), RGB145.1 (VDD), RGB146.1 (VDD), RGB147.1 (VDD), RGB148.1 (VDD), RGB149.1 (VDD), RGB150.1 (VDD), RGB151.1 (VDD), RGB152.1 (VDD); no longer R20.1, R21.1, R22.1, R23.1, R24.1, R25.1, R26.1, R27.1, R28.1
- net GND: now also C100.2, C135.2, C136.2, C137.2, C138.2, C139.2, C140.2, C141.2, C58.2, C59.2, C60.2, C61.2, C62.2, C63.2, C64.2, C65.2, C66.2, C67.2, C68.2, C69.2, C70.2, C71.2, C72.2, C73.2, C74.2, C75.2, C76.2, C77.2, C78.2, C79.2, C82.2, C83.2, C84.2, C85.2, C86.2, C87.2, C88.2, C89.2, C90.2, C91.2, C92.2, C93.2, C94.2, C95.2, C96.2, C97.2, C98.2, C99.2, RGB106.3 (VSS), RGB107.3 (VSS), RGB108.3 (VSS), RGB109.3 (VSS), RGB110.3 (VSS), RGB111.3 (VSS), RGB112.3 (VSS), RGB113.3 (VSS), RGB114.3 (VSS), RGB115.3 (VSS), RGB116.3 (VSS), RGB117.3 (VSS), RGB118.3 (VSS), RGB119.3 (VSS), RGB120.3 (VSS), RGB121.3 (VSS), RGB122.3 (VSS), RGB123.3 (VSS), RGB124.3 (VSS), RGB125.3 (VSS), RGB126.3 (VSS), RGB127.3 (VSS), RGB128.3 (VSS), RGB129.3 (VSS), RGB130.3 (VSS), RGB131.3 (VSS), RGB132.3 (VSS), RGB133.3 (VSS), RGB134.3 (VSS), RGB135.3 (VSS), RGB136.3 (VSS), RGB137.3 (VSS), RGB138.3 (VSS), RGB139.3 (VSS), RGB140.3 (VSS), RGB141.3 (VSS), RGB142.3 (VSS), RGB143.3 (VSS), RGB144.3 (VSS), RGB145.3 (VSS), RGB146.3 (VSS), RGB147.3 (VSS), RGB148.3 (VSS), RGB149.3 (VSS), RGB150.3 (VSS), RGB151.3 (VSS), RGB152.3 (VSS)
- net at RGB105.2 (DOUT): now also RGB106.4 (DIN)
- net COL_0_R renamed COL0
- net COL_1_R renamed COL1
- net COL_2_R renamed COL2
- net COL_3_R renamed COL3
- net COL_4_R renamed COL4
- net COL_5_R renamed COL5
- net COL_6_R renamed COL6
- net COL_7_R renamed COL7
- net COL_8_R renamed COL8
- net COL8: now also RE1.S2, C137.1; no longer RE1.S1
- net RE_1_A renamed RE_A
- net RE_A: now also C136.1, R56.1; no longer C81.1
- net RE_1_B renamed RE_B
- net RE_B: now also C135.1, R55.1; no longer C80.1
- net RE_SW2: no longer names the net of D51.2 (A)
- net RE_SW2: now also RE1.S1; no longer RE1.S2
- net RGB_IN_R renamed RGB_IN
- net ROW_0_R renamed ROW0
- net ROW_1_R renamed ROW1
- net ROW_2_R renamed ROW2
- net ROW_3_R renamed ROW3
- net ROW_4_R renamed ROW4
- net ROW_5_R renamed ROW5
- new net: RGB132.2 (DOUT), RGB134.4 (DIN)
- new net: RGB130.2 (DOUT), RGB132.4 (DIN)
- new net: RGB121.2 (DOUT), RGB123.4 (DIN)
- new net: RGB119.2 (DOUT), RGB121.4 (DIN)
- new net: RGB115.2 (DOUT), RGB116.4 (DIN)
- new net: RGB114.2 (DOUT), RGB115.4 (DIN)
- new net: RGB106.2 (DOUT), RGB107.4 (DIN)
- new net: RGB140.2 (DOUT), RGB142.4 (DIN)
- new net: RGB138.2 (DOUT), RGB140.4 (DIN)
- new net: RGB113.2 (DOUT), RGB114.4 (DIN)
- new net: RGB130.4 (DIN), RGB151.2 (DOUT)
- new net: RGB149.2 (DOUT), RGB151.4 (DIN)
- new net: RGB146.2 (DOUT), RGB148.4 (DIN)
- new net: RGB144.2 (DOUT), RGB146.4 (DIN)
- new net: RGB123.2 (DOUT), RGB125.4 (DIN)
- new net: RGB111.2 (DOUT), RGB112.4 (DIN)
- new net: RGB110.2 (DOUT), RGB111.4 (DIN)
- new net: RGB150.2 (DOUT), RGB152.4 (DIN)
- new net: RGB148.2 (DOUT), RGB150.4 (DIN)
- new net: RGB125.2 (DOUT), RGB127.4 (DIN)
- new net: RGB118.4 (DIN), RGB127.2 (DOUT)
- new net: RGB126.2 (DOUT), RGB128.4 (DIN)
- new net: RGB124.2 (DOUT), RGB126.4 (DIN)
- new net: RGB117.2 (DOUT), RGB119.4 (DIN)
- new net: RGB109.2 (DOUT), RGB110.4 (DIN)
- new net: RGB118.2 (DOUT), RGB120.4 (DIN)
- new net: RGB122.2 (DOUT), RGB124.4 (DIN)
- new net: RGB120.2 (DOUT), RGB122.4 (DIN)
- new net: RGB116.2 (DOUT), RGB117.4 (DIN)
- new net: RGB142.2 (DOUT), RGB144.4 (DIN)
- new net: RGB133.2 (DOUT), RGB135.4 (DIN)
- new net: RGB131.2 (DOUT), RGB133.4 (DIN)
- new net: RGB137.2 (DOUT), RGB139.4 (DIN)
- new net: RGB135.2 (DOUT), RGB137.4 (DIN)
- new net: RGB129.2 (DOUT), RGB131.4 (DIN)
- new net: RGB112.2 (DOUT), RGB113.4 (DIN)
- new net: RGB139.2 (DOUT), RGB141.4 (DIN)
- new net: RGB108.2 (DOUT), RGB109.4 (DIN)
- new net: RGB107.2 (DOUT), RGB108.4 (DIN)
- new net: RGB147.2 (DOUT), RGB149.4 (DIN)
- new net: RGB128.2 (DOUT), RGB129.4 (DIN)
- new net: RGB136.2 (DOUT), RGB138.4 (DIN)
- new net: RGB134.2 (DOUT), RGB136.4 (DIN)
- new net: RGB145.2 (DOUT), RGB147.4 (DIN)
- new net: RGB143.2 (DOUT), RGB145.4 (DIN)
- new net: RGB141.2 (DOUT), RGB143.4 (DIN)
- new net +3V3: R20.1, R21.1, R22.1, R23.1, R24.1, R25.1, R26.1, R27.1, R28.1, R55.2, R56.2
- new net RGB_OUT: RGB152.2 (DOUT)
Other:
- note added: "LED matrix"
- note added: "Rotary encoder"
- note added: "Switch matrix"
- moved on the sheet: C57, D43, D44, D45, D46, D47, D48, D49, D50, D51, D52, D53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

Commit message: layout improvements
Parts:
- C47: renamed from C57; footprint Capacitor_SMD:C_0805_2012Metric -> Capacitor_SMD:C_0603_1608Metric
- C48: renamed from C58; footprint Capacitor_SMD:C_0805_2012Metric -> Capacitor_SMD:C_0603_1608Metric
- C49: renamed from C59; footprint Capacitor_SMD:C_0805_2012Metric -> Capacitor_SMD:C_0603_1608Metric
- C50: renamed from C60; footprint Capacitor_SMD:C_0805_2012Metric -> Capacitor_SMD:C_0603_1608Metric
- C51: renamed from C61; footprint Capacitor_SMD:C_0805_2012Metric -> Capacitor_SMD:C_0603_1608Metric
- C52: renamed from C62; footprint Capacitor_SMD:C_0805_2012Metric -> Capacitor_SMD:C_0603_1608Metric
- C53: renamed from C63; footprint Capacitor_SMD:C_0805_2012Metric -> Capacitor_SMD:C_0603_1608Metric
- C54: renamed from C64; footprint Capacitor_SMD:C_0805_2012Metric -> Capacitor_SMD:C_0603_1608Metric
- C55: renamed from C65; footprint Capacitor_SMD:C_0805_2012Metric -> Capacitor_SMD:C_0603_1608Metric
- C56: renamed from C66; footprint Capacitor_SMD:C_0805_2012Metric -> Capacitor_SMD:C_0603_1608Metric
- C57: renamed from C67; footprint Capacitor_SMD:C_0805_2012Metric -> Capacitor_SMD:C_0603_1608Metric
- C58: renamed from C68; footprint Capacitor_SMD:C_0805_2012Metric -> Capacitor_SMD:C_0603_1608Metric
- C59: renamed from C69; footprint Capacitor_SMD:C_0805_2012Metric -> Capacitor_SMD:C_0603_1608Metric
- C60: renamed from C71; footprint Capacitor_SMD:C_0805_2012Metric -> Capacitor_SMD:C_0603_1608Metric
- C61: renamed from C73; footprint Capacitor_SMD:C_0805_2012Metric -> Capacitor_SMD:C_0603_1608Metric
- C62: renamed from C75; footprint Capacitor_SMD:C_0805_2012Metric -> Capacitor_SMD:C_0603_1608Metric
- C63: renamed from C77; footprint Capacitor_SMD:C_0805_2012Metric -> Capacitor_SMD:C_0603_1608Metric
- C64: renamed from C79; footprint Capacitor_SMD:C_0805_2012Metric -> Capacitor_SMD:C_0603_1608Metric
- C65: renamed from C70; footprint Capacitor_SMD:C_0805_2012Metric -> Capacitor_SMD:C_0603_1608Metric
- C66: renamed from C72; footprint Capacitor_SMD:C_0805_2012Metric -> Capacitor_SMD:C_0603_1608Metric
- C67: renamed from C74; footprint Capacitor_SMD:C_0805_2012Metric -> Capacitor_SMD:C_0603_1608Metric
- C68: renamed from C76; footprint Capacitor_SMD:C_0805_2012Metric -> Capacitor_SMD:C_0603_1608Metric
- C69: renamed from C78; footprint Capacitor_SMD:C_0805_2012Metric -> Capacitor_SMD:C_0603_1608Metric
- C70: renamed from C80; footprint Capacitor_SMD:C_0805_2012Metric -> Capacitor_SMD:C_0603_1608Metric
- C71: renamed from C81; footprint Capacitor_SMD:C_0805_2012Metric -> Capacitor_SMD:C_0603_1608Metric
- C72: renamed from C83; footprint Capacitor_SMD:C_0805_2012Metric -> Capacitor_SMD:C_0603_1608Metric
- C73: renamed from C85; footprint Capacitor_SMD:C_0805_2012Metric -> Capacitor_SMD:C_0603_1608Metric
- C74: renamed from C87; footprint Capacitor_SMD:C_0805_2012Metric -> Capacitor_SMD:C_0603_1608Metric
- C75: renamed from C89; footprint Capacitor_SMD:C_0805_2012Metric -> Capacitor_SMD:C_0603_1608Metric
- C76: renamed from C91; footprint Capacitor_SMD:C_0805_2012Metric -> Capacitor_SMD:C_0603_1608Metric
- C77: renamed from C93; footprint Capacitor_SMD:C_0805_2012Metric -> Capacitor_SMD:C_0603_1608Metric
- C78: renamed from C95; footprint Capacitor_SMD:C_0805_2012Metric -> Capacitor_SMD:C_0603_1608Metric
- C79: renamed from C97; footprint Capacitor_SMD:C_0805_2012Metric -> Capacitor_SMD:C_0603_1608Metric
- C80: renamed from C99; footprint Capacitor_SMD:C_0805_2012Metric -> Capacitor_SMD:C_0603_1608Metric
- C81: renamed from C138; footprint Capacitor_SMD:C_0805_2012Metric -> Capacitor_SMD:C_0603_1608Metric
- C82: renamed from C140; footprint Capacitor_SMD:C_0805_2012Metric -> Capacitor_SMD:C_0603_1608Metric
- C83: renamed from C82; footprint Capacitor_SMD:C_0805_2012Metric -> Capacitor_SMD:C_0603_1608Metric
- C84: footprint Capacitor_SMD:C_0805_2012Metric -> Capacitor_SMD:C_0603_1608Metric
- C85: renamed from C86; footprint Capacitor_SMD:C_0805_2012Metric -> Capacitor_SMD:C_0603_1608Metric
- C86: renamed from C88; footprint Capacitor_SMD:C_0805_2012Metric -> Capacitor_SMD:C_0603_1608Metric
- C87: renamed from C90; footprint Capacitor_SMD:C_0805_2012Metric -> Capacitor_SMD:C_0603_1608Metric
- C88: renamed from C92; footprint Capacitor_SMD:C_0805_2012Metric -> Capacitor_SMD:C_0603_1608Metric
- C89: renamed from C94; footprint Capacitor_SMD:C_0805_2012Metric -> Capacitor_SMD:C_0603_1608Metric
- C90: renamed from C96; footprint Capacitor_SMD:C_0805_2012Metric -> Capacitor_SMD:C_0603_1608Metric
- C91: renamed from C98; footprint Capacitor_SMD:C_0805_2012Metric -> Capacitor_SMD:C_0603_1608Metric
- C92: renamed from C100; footprint Capacitor_SMD:C_0805_2012Metric -> Capacitor_SMD:C_0603_1608Metric
- C93: renamed from C139; footprint Capacitor_SMD:C_0805_2012Metric -> Capacitor_SMD:C_0603_1608Metric
- C94: renamed from C141; footprint Capacitor_SMD:C_0805_2012Metric -> Capacitor_SMD:C_0603_1608Metric
- R19: renamed from R20; footprint Resistor_SMD:R_0805_2012Metric -> Resistor_SMD:R_0603_1608Metric
- R20: renamed from R21; footprint Resistor_SMD:R_0805_2012Metric -> Resistor_SMD:R_0603_1608Metric
- R21: renamed from R22; footprint Resistor_SMD:R_0805_2012Metric -> Resistor_SMD:R_0603_1608Metric
- R22: renamed from R23; footprint Resistor_SMD:R_0805_2012Metric -> Resistor_SMD:R_0603_1608Metric
- R23: renamed from R24; footprint Resistor_SMD:R_0805_2012Metric -> Resistor_SMD:R_0603_1608Metric
- R24: renamed from R25; footprint Resistor_SMD:R_0805_2012Metric -> Resistor_SMD:R_0603_1608Metric
- R25: renamed from R26; footprint Resistor_SMD:R_0805_2012Metric -> Resistor_SMD:R_0603_1608Metric
- R26: renamed from R27; footprint Resistor_SMD:R_0805_2012Metric -> Resistor_SMD:R_0603_1608Metric
- R27: renamed from R28; footprint Resistor_SMD:R_0805_2012Metric -> Resistor_SMD:R_0603_1608Metric
- RGB37: renamed from RGB105; footprint LED_SMD:LED_WS2812B_PLCC4_5.0x5.0mm_P3.2mm -> mechpad:6028_LED
- RGB38: renamed from RGB106; footprint LED_SMD:LED_WS2812B_PLCC4_5.0x5.0mm_P3.2mm -> mechpad:6028_LED
- RGB39: renamed from RGB107; footprint LED_SMD:LED_WS2812B_PLCC4_5.0x5.0mm_P3.2mm -> mechpad:6028_LED
- RGB40: renamed from RGB108; footprint LED_SMD:LED_WS2812B_PLCC4_5.0x5.0mm_P3.2mm -> mechpad:6028_LED
- RGB41: renamed from RGB109; footprint LED_SMD:LED_WS2812B_PLCC4_5.0x5.0mm_P3.2mm -> mechpad:6028_LED
- RGB42: renamed from RGB110; footprint LED_SMD:LED_WS2812B_PLCC4_5.0x5.0mm_P3.2mm -> mechpad:6028_LED
- RGB43: renamed from RGB111; footprint LED_SMD:LED_WS2812B_PLCC4_5.0x5.0mm_P3.2mm -> mechpad:6028_LED
- RGB44: renamed from RGB112; footprint LED_SMD:LED_WS2812B_PLCC4_5.0x5.0mm_P3.2mm -> mechpad:6028_LED
- RGB45: renamed from RGB113; footprint LED_SMD:LED_WS2812B_PLCC4_5.0x5.0mm_P3.2mm -> mechpad:6028_LED
- RGB46: renamed from RGB114; footprint LED_SMD:LED_WS2812B_PLCC4_5.0x5.0mm_P3.2mm -> mechpad:6028_LED
- RGB47: renamed from RGB115; footprint LED_SMD:LED_WS2812B_PLCC4_5.0x5.0mm_P3.2mm -> mechpad:6028_LED
- RGB48: renamed from RGB116; footprint LED_SMD:LED_WS2812B_PLCC4_5.0x5.0mm_P3.2mm -> mechpad:6028_LED
- RGB49: renamed from RGB117; footprint LED_SMD:LED_WS2812B_PLCC4_5.0x5.0mm_P3.2mm -> mechpad:6028_LED
- RGB50: renamed from RGB119; footprint LED_SMD:LED_WS2812B_PLCC4_5.0x5.0mm_P3.2mm -> mechpad:6028_LED
- RGB51: renamed from RGB121; footprint LED_SMD:LED_WS2812B_PLCC4_5.0x5.0mm_P3.2mm -> mechpad:6028_LED
- RGB52: renamed from RGB123; footprint LED_SMD:LED_WS2812B_PLCC4_5.0x5.0mm_P3.2mm -> mechpad:6028_LED
- RGB53: renamed from RGB125; footprint LED_SMD:LED_WS2812B_PLCC4_5.0x5.0mm_P3.2mm -> mechpad:6028_LED
- RGB54: renamed from RGB127; footprint LED_SMD:LED_WS2812B_PLCC4_5.0x5.0mm_P3.2mm -> mechpad:6028_LED
- RGB55: renamed from RGB118; footprint LED_SMD:LED_WS2812B_PLCC4_5.0x5.0mm_P3.2mm -> mechpad:6028_LED
- RGB56: renamed from RGB120; footprint LED_SMD:LED_WS2812B_PLCC4_5.0x5.0mm_P3.2mm -> mechpad:6028_LED
- RGB57: renamed from RGB122; footprint LED_SMD:LED_WS2812B_PLCC4_5.0x5.0mm_P3.2mm -> mechpad:6028_LED
- RGB58: renamed from RGB124; footprint LED_SMD:LED_WS2812B_PLCC4_5.0x5.0mm_P3.2mm -> mechpad:6028_LED
- RGB59: renamed from RGB126; footprint LED_SMD:LED_WS2812B_PLCC4_5.0x5.0mm_P3.2mm -> mechpad:6028_LED
- RGB60: renamed from RGB128; footprint LED_SMD:LED_WS2812B_PLCC4_5.0x5.0mm_P3.2mm -> mechpad:6028_LED
- RGB61: renamed from RGB129; footprint LED_SMD:LED_WS2812B_PLCC4_5.0x5.0mm_P3.2mm -> mechpad:6028_LED
- RGB62: renamed from RGB131; footprint LED_SMD:LED_WS2812B_PLCC4_5.0x5.0mm_P3.2mm -> mechpad:6028_LED
- RGB63: renamed from RGB133; footprint LED_SMD:LED_WS2812B_PLCC4_5.0x5.0mm_P3.2mm -> mechpad:6028_LED
- RGB64: renamed from RGB135; footprint LED_SMD:LED_WS2812B_PLCC4_5.0x5.0mm_P3.2mm -> mechpad:6028_LED
- RGB65: renamed from RGB137; footprint LED_SMD:LED_WS2812B_PLCC4_5.0x5.0mm_P3.2mm -> mechpad:6028_LED
- RGB66: renamed from RGB139; footprint LED_SMD:LED_WS2812B_PLCC4_5.0x5.0mm_P3.2mm -> mechpad:6028_LED
- RGB67: renamed from RGB141; footprint LED_SMD:LED_WS2812B_PLCC4_5.0x5.0mm_P3.2mm -> mechpad:6028_LED
- RGB68: renamed from RGB143; footprint LED_SMD:LED_WS2812B_PLCC4_5.0x5.0mm_P3.2mm -> mechpad:6028_LED
- RGB69: renamed from RGB145; footprint LED_SMD:LED_WS2812B_PLCC4_5.0x5.0mm_P3.2mm -> mechpad:6028_LED
- RGB70: renamed from RGB147; footprint LED_SMD:LED_WS2812B_PLCC4_5.0x5.0mm_P3.2mm -> mechpad:6028_LED
- RGB71: renamed from RGB149; footprint LED_SMD:LED_WS2812B_PLCC4_5.0x5.0mm_P3.2mm -> mechpad:6028_LED
- RGB72: renamed from RGB151; footprint LED_SMD:LED_WS2812B_PLCC4_5.0x5.0mm_P3.2mm -> mechpad:6028_LED
- RGB73: renamed from RGB130; footprint LED_SMD:LED_WS2812B_PLCC4_5.0x5.0mm_P3.2mm -> mechpad:6028_LED
- RGB74: renamed from RGB132; footprint LED_SMD:LED_WS2812B_PLCC4_5.0x5.0mm_P3.2mm -> mechpad:6028_LED
- RGB75: renamed from RGB134; footprint LED_SMD:LED_WS2812B_PLCC4_5.0x5.0mm_P3.2mm -> mechpad:6028_LED
- RGB76: renamed from RGB136; footprint LED_SMD:LED_WS2812B_PLCC4_5.0x5.0mm_P3.2mm -> mechpad:6028_LED
- RGB77: renamed from RGB138; footprint LED_SMD:LED_WS2812B_PLCC4_5.0x5.0mm_P3.2mm -> mechpad:6028_LED
- RGB78: renamed from RGB140; footprint LED_SMD:LED_WS2812B_PLCC4_5.0x5.0mm_P3.2mm -> mechpad:6028_LED
- RGB79: renamed from RGB142; footprint LED_SMD:LED_WS2812B_PLCC4_5.0x5.0mm_P3.2mm -> mechpad:6028_LED
- RGB80: renamed from RGB144; footprint LED_SMD:LED_WS2812B_PLCC4_5.0x5.0mm_P3.2mm -> mechpad:6028_LED
- RGB81: renamed from RGB146; footprint LED_SMD:LED_WS2812B_PLCC4_5.0x5.0mm_P3.2mm -> mechpad:6028_LED
- RGB82: renamed from RGB148; footprint LED_SMD:LED_WS2812B_PLCC4_5.0x5.0mm_P3.2mm -> mechpad:6028_LED
- RGB83: renamed from RGB150; footprint LED_SMD:LED_WS2812B_PLCC4_5.0x5.0mm_P3.2mm -> mechpad:6028_LED
- RGB84: renamed from RGB152; footprint LED_SMD:LED_WS2812B_PLCC4_5.0x5.0mm_P3.2mm -> mechpad:6028_LED
- renumbered C137 to C44, C135 to C45, C136 to C46, D43 to D40, D44 to D41, D45 to D42, D46 to D43, D47 to D44, D48 to D45, D49 to D46, D50 to D47, D51 to D48, D52 to D49, D53 to D50, D54 to D51, D55 to D52, D56 to D53, D57 to D54, D58 to D55, D59 to D56, D60 to D57, D61 to D58, D62 to D59, D63 to D60, D64 to D61, D65 to D62, D66 to D63, D67 to D64, D68 to D65, D69 to D66, D70 to D67, D71 to D68, D72 to D69, D73 to D70, D74 to D71, D75 to D72, D76 to D73, D77 to D74, D78 to D75, D79 to D76, D80 to D77, D81 to D78, D82 to D79, D83 to D80, D84 to D81, D85 to D82, D86 to D83, D87 to D84, D88 to D85, D89 to D86, D90 to D87, D91 to D88, R55 to R28, R56 to R29, SW38 to SW37, SW39 to SW38, SW40 to SW39, SW41 to SW40, SW42 to SW41, SW43 to SW42, SW44 to SW43, SW45 to SW44, SW46 to SW45, SW47 to SW46, SW48 to SW47, SW49 to SW48, SW50 to SW49, SW51 to SW50, SW52 to SW51, SW53 to SW52, SW54 to SW53, SW55 to SW54, SW56 to SW55, SW57 to SW56, SW58 to SW57, SW59 to SW58, SW60 to SW59, SW61 to SW60, SW62 to SW61, SW63 to SW62, SW64 to SW63, SW65 to SW64, SW66 to SW65, SW67 to SW66, SW68 to SW67, SW69 to SW68, SW70 to SW69, SW71 to SW70, SW72 to SW71, SW73 to SW72, SW74 to SW73, SW75 to SW74, SW76 to SW75, SW77 to SW76, SW78 to SW77, SW79 to SW78, SW80 to SW79, SW81 to SW80, SW82 to SW81, SW83 to SW82, SW84 to SW83, SW85 to SW84
