File: Schematics and PCB/Schematics and PCB.kicad_pcb (KiCad board)
At the start: 2 copper layers, 512 parts, among them Q1 FDN340P, Q2 FDN340P, Q3 FDN340P, Q4 FS8205, SW10 1, SW100 NUMPAD15, SW101 NUMPAD16, SW102 NUMPAD17, SW103 NUMPAD18, SW104 NUMPAD19, SW105 NUMPAD20, SW108 Battery Switch, SW11 2, SW12 3, SW13 4, SW14 5, SW15 6, SW16 TAB, SW17 Q, SW18 W, SW19 E, SW2 ESC, SW20 R, SW21 T, SW22 MAYUS, SW23 A, SW24 S, SW25 D, SW26 F, SW27 G, SW28 L_SHIFT, SW29 Z, SW3 F1, SW30 X, SW31 C, SW32 V, SW33 B, SW34 L_CRTL, SW35 OS, SW36 L_ALT, SW37 L_SPACE, SW38 F7, SW39 F8, SW4 F2, SW40 F9, SW41 F10, SW42 F11, SW43 F12, SW44 PRT_SCR, SW45 DEL, SW46 7, SW47 8, SW48 9, SW49 0, SW5 F3, SW50 -, SW51 =, SW52 BACKSPACE, SW53 MACRO1, SW54 Y, SW55 U, SW56 I, SW57 O, SW58 P, SW59 [, SW6 F4, SW60 ], SW61 \, SW62 MACRO2, SW63 H, SW64 J, SW65 K, SW66 L, SW67 ;, SW68 ', SW69 ENTER, SW7 F5, SW70 MACRO3, SW71 N, SW72 M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

Commit message: Finished initial iteration of the Right layout
Parts:
- removed the D51 at (318.7, -241.2)
- removed the D59 at (324.5, -247.9)
- removed the D68 at (330.3, -251.3)
- removed the D76 at (336.1, -258.0)
- removed the D84 at (341.9, -264.7)
- removed the SW62 at (208.3, 87.6)
- removed the SW70 at (208.3, 106.7)
- removed the SW78 at (208.3, 125.7)
- added D58: 1N4148W, Diode_SMD:D_SOD-123, F.Cu at (202.6, 67.7)
- added D74: 1N4148W, Diode_SMD:D_SOD-123, F.Cu at (202.6, 86.7)
- added D82: 1N4148W, Diode_SMD:D_SOD-123, F.Cu at (202.6, 105.8)
- added D90: 1N4148W, Diode_SMD:D_SOD-123, F.Cu at (219.1, 124.8)
- added J11: Conn_01x12, Connector_FFC-FPC:Hirose_FH12-12S-0.5SH_1x12-1MP_P0.50mm_Horizontal, B.Cu at (67.1, 56.0)
- added SW69: MACRO2, Button_Switch_Keyboard:SW_Cherry_MX_1.00u_PCB, F.Cu at (208.3, 87.6)
- added SW77: MACRO3, Button_Switch_Keyboard:SW_Cherry_MX_1.00u_PCB, F.Cu at (208.3, 106.7)
- added SW85: MACRO4, Button_Switch_Keyboard:SW_Cherry_MX_1.00u_PCB, F.Cu at (208.3, 125.7)
- added U18: TLV71311PDBVR, Package_TO_SOT_SMD:TSOT-23-5, F.Cu at (509.7, -136.0)
- added U19: TLV70033DDCR, Package_TO_SOT_SMD:TSOT-23-5, F.Cu at (509.7, -131.5)
- added U6: ~, Package_SO:SOP-16_3.9x9.9mm_P1.27mm, B.Cu at (59.3, 139.7)
- added U7: 74HC165, Package_SO:SOP-16_3.9x9.9mm_P1.27mm, B.Cu at (96.0, 140.3)
- C100: renamed from C88; moved to B.Cu
- C101: renamed from C89; moved to B.Cu
- R20, R21, R22, R23, R24, R25, R26, R27, R29, R30: moved to B.Cu
- R28: value 10K -> 10k; footprint Resistor_SMD:R_0805_2012Metric -> Resistor_SMD:R_0603_1608Metric; moved to B.Cu
- moved RGB69 551.1 mm to (53.6, 95.2)
- moved RGB71 542.7 mm to (82.2, 114.3), turned to 180 degrees
- moved RGB83 532.6 mm to (115.6, 133.3)
- moved RGB70 529.6 mm to (63.1, 114.3), turned to 180 degrees
- moved RGB81 526.6 mm to (153.7, 133.3)
- moved RGB53 523.0 mm to (48.9, 76.2), turned to 180 degrees
- moved RGB78 522.7 mm to (210.8, 133.3)
- moved RGB79 522.3 mm to (191.8, 133.3)
- moved RGB68 518.5 mm to (72.6, 95.2)
- moved RGB84 517.1 mm to (77.5, 133.3)
- moved RGB74 511.4 mm to (139.3, 114.3), turned to 180 degrees
- moved RGB76 501.5 mm to (191.8, 114.3), turned to 180 degrees
- moved RGB54 501.5 mm to (67.9, 76.2), turned to 180 degrees
- moved RGB72 500.5 mm to (101.2, 114.3), turned to 180 degrees
- moved RGB82 500.5 mm to (134.6, 133.3)
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- renumbered C207 to C211, C210 to C212, C211 to C213, C215 to C52, C52 to C53, C53 to C54, C54 to C55, C55 to C56, C56 to C57, C57 to C58, C58 to C59, C59 to C60, C60 to C61, C61 to C62, C62 to C63, C63 to C64, C64 to C65, C65 to C66, C66 to C67, C67 to C68, C68 to C69, C69 to C70, C70 to C71, C71 to C72, C72 to C73, C73 to C74, C74 to C75, C75 to C76, C79 to C77, C83 to C78, C87 to C79, C93 to C80, C97 to C81, C76 to C82, C80 to C83, C90 to C85, C94 to C86, C98 to C87, C77 to C88, C81 to C89, C85 to C90, C95 to C92, C99 to C93, C78 to C94, C82 to C95, C86 to C96, C92 to C97, C96 to C98, C100 to C99, D101 to D100, D102 to D101, D103 to D102, D104 to D103, D105 to D104, D106 to D105, D107 to D106, D108 to D107, D109 to D108, D110 to D109, D111 to D110, D112 to D111, D113 to D112, D114 to D113, D115 to D114, D128 to D127, D129 to D128, D130 to D129, D52 to D51, D53 to D52, D54 to D53, D55 to D54, D56 to D55, D57 to D56, D58 to D57, D60 to D59, D61 to D60, D62 to D61, D63 to D62, D64 to D63, D65 to D64, D66 to D65, D67 to D66, D69 to D67, D70 to D68, D71 to D69, D72 to D70, D73 to D71, D74 to D72, D75 to D73, D77 to D75, D78 to D76, D79 to D77, D80 to D78, D81 to D79, D82 to D80, D83 to D81, D85 to D83, D86 to D84, D87 to D85, D88 to D86, D89 to D87, D90 to D88, D91 to D89, D92 to D91, D93 to D92, D94 to D93, D95 to D94, D96 to D95, D97 to D96, D98 to D97, D99 to D98, D100 to D99, R105 to R103, R106 to R104, R107 to R105, R108 to R106, R109 to R107, R110 to R108, R112 to R110, R113 to R111, R33 to R31, R34 to R32, R35 to R33, R36 to R34, R37 to R35, R38 to R36, R39 to R37, R40 to R38, R41 to R39, R42 to R40, R43 to R41, R44 to R42, R45 to R43, R46 to R44, R47 to R45, R48 to R46, R49 to R47, R50 to R48, R51 to R49, R52 to R50, R53 to R51, R65 to R63, R77 to R79, R86 to R84, R92 to R90, R93 to R91, R99 to R97, RGB105 to RGB37, RGB37 to RGB38, RGB38 to RGB39, RGB39 to RGB40, RGB40 to RGB41, RGB41 to RGB42, RGB42 to RGB43, RGB43 to RGB44, RGB44 to RGB45, RGB45 to RGB46, RGB46 to RGB47, RGB47 to RGB48, RGB48 to RGB49, RGB52 to RGB51, RGB54 to RGB52, RGB56 to RGB53, RGB58 to RGB54, RGB59 to RGB55, RGB57 to RGB56, RGB55 to RGB57, RGB53 to RGB58, RGB51 to RGB59, RGB49 to RGB60, RGB60 to RGB61, RGB64 to RGB62, RGB68 to RGB63, RGB72 to RGB64, RGB76 to RGB65, RGB80 to RGB66, RGB81 to RGB67, RGB77 to RGB68, RGB73 to RGB69, RGB69 to RGB70, RGB65 to RGB71, RGB61 to RGB72, RGB62 to RGB73, RGB66 to RGB74, RGB70 to RGB75, RGB74 to RGB76, RGB78 to RGB77, RGB82 to RGB78, RGB83 to RGB79, RGB79 to RGB80, RGB75 to RGB81, RGB71 to RGB82, RGB67 to RGB83, RGB63 to RGB84, SW63 to SW62, SW64 to SW63, SW65 to SW64, SW66 to SW65, SW67 to SW66, SW68 to SW67, SW69 to SW68, SW71 to SW70, SW72 to SW71, SW73 to SW72, SW74 to SW73, SW75 to SW74, SW76 to SW75, SW77 to SW76, SW79 to SW78, SW80 to SW79, SW81 to SW80, SW82 to SW81, SW83 to SW82, SW84 to SW83, SW85 to SW84, U10 to U11, U11 to U12, U12 to U13, U14 to U15, U18 to U17, U19 to U20, U20 to U21, U24 to U23, U7 to U8, U8 to U9
Connections:
- net /Li-Po Charge Boost/5V_IN renamed /V_USB
- C100 pad 1: /Main IC1/D11# -> /RE_1_B
- C101 pad 1: /Main IC1/D10# -> /RE_1_A
- D43 pad 1: /Main IC1/A0 -> /Right Switch Matrix/ROW_0_R
- D44 pad 1: /Main IC1/A0 -> /Right Switch Matrix/ROW_0_R
- D45 pad 1: /Main IC1/A0 -> /Right Switch Matrix/ROW_0_R
- D46 pad 1: /Main IC1/A0 -> /Right Switch Matrix/ROW_0_R
- D47 pad 1: /Main IC1/A0 -> /Right Switch Matrix/ROW_0_R
- D48 pad 1: /Main IC1/A0 -> /Right Switch Matrix/ROW_0_R
- D49 pad 1: /Main IC1/A0 -> /Right Switch Matrix/ROW_0_R
- D50 pad 1: /Main IC1/A0 -> /Right Switch Matrix/ROW_0_R
- D51 pad 1: /Main IC1/A1 -> /Right Switch Matrix/ROW_1_R
- D52 pad 1: /Main IC1/A1 -> /Right Switch Matrix/ROW_1_R
- D53 pad 1: /Main IC1/A1 -> /Right Switch Matrix/ROW_1_R
- D54 pad 1: /Main IC1/A1 -> /Right Switch Matrix/ROW_1_R
- D55 pad 1: /Main IC1/A1 -> /Right Switch Matrix/ROW_1_R
- D56 pad 1: /Main IC1/A1 -> /Right Switch Matrix/ROW_1_R
- D57 pad 1: /Main IC1/A1 -> /Right Switch Matrix/ROW_1_R
- D59 pad 1: /Main IC1/A2 -> /Right Switch Matrix/ROW_2_R
- D60 pad 1: /Main IC1/A2 -> /Right Switch Matrix/ROW_2_R
- D61 pad 1: /Main IC1/A2 -> /Right Switch Matrix/ROW_2_R
- D62 pad 1: /Main IC1/A2 -> /Right Switch Matrix/ROW_2_R
- D63 pad 1: /Main IC1/A2 -> /Right Switch Matrix/ROW_2_R
- D64 pad 1: /Main IC1/A2 -> /Right Switch Matrix/ROW_2_R
- D65 pad 1: /Main IC1/A2 -> /Right Switch Matrix/ROW_2_R
- D66 pad 1: /Main IC1/A2 -> /Right Switch Matrix/ROW_2_R
- D67 pad 1: /Main IC1/A3 -> /Right Switch Matrix/ROW_3_R
- D68 pad 1: /Main IC1/A3 -> /Right Switch Matrix/ROW_3_R
- D69 pad 1: /Main IC1/A3 -> /Right Switch Matrix/ROW_3_R
- D70 pad 1: /Main IC1/A3 -> /Right Switch Matrix/ROW_3_R
- D71 pad 1: /Main IC1/A3 -> /Right Switch Matrix/ROW_3_R
- D72 pad 1: /Main IC1/A3 -> /Right Switch Matrix/ROW_3_R
- D73 pad 1: /Main IC1/A3 -> /Right Switch Matrix/ROW_3_R
- D75 pad 1: /Main IC1/A4 -> /Right Switch Matrix/ROW_4_R
- D76 pad 1: /Main IC1/A4 -> /Right Switch Matrix/ROW_4_R
- D77 pad 1: /Main IC1/A4 -> /Right Switch Matrix/ROW_4_R
- D78 pad 1: /Main IC1/A4 -> /Right Switch Matrix/ROW_4_R
- D79 pad 1: /Main IC1/A4 -> /Right Switch Matrix/ROW_4_R
- D80 pad 1: /Main IC1/A4 -> /Right Switch Matrix/ROW_4_R
- D81 pad 1: /Main IC1/A4 -> /Right Switch Matrix/ROW_4_R
- D83 pad 1: /Main IC1/A5 -> /Right Switch Matrix/ROW_5_R
- D84 pad 1: /Main IC1/A5 -> /Right Switch Matrix/ROW_5_R
- D85 pad 1: /Main IC1/A5 -> /Right Switch Matrix/ROW_5_R
- D86 pad 1: /Main IC1/A5 -> /Right Switch Matrix/ROW_5_R
- D87 pad 1: /Main IC1/A5 -> /Right Switch Matrix/ROW_5_R
- D88 pad 1: /Main IC1/A5 -> /Right Switch Matrix/ROW_5_R
- D89 pad 1: /Main IC1/A5 -> /Right Switch Matrix/ROW_5_R
- R20 pad 2: /Main IC1/D4 -> /Right Switch Matrix/COL_0_R
- R28 pad 2: /Right Switch Matrix/RE_SW1 -> /RE_SW
- R29 pad 2: /Main IC1/D11# -> /RE_1_B
- R30 pad 2: /Main IC1/D10# -> /RE_1_A
- RE1 pad A: /Main IC1/D11# -> /RE_1_B
- RE1 pad B: /Main IC1/D10# -> /RE_1_A
- RE1 pad S1: /Right Switch Matrix/RE_SW1 -> /RE_SW
- RE1 pad S2: /Right Switch Matrix/RE_SW2 -> GND
- RGB37 pad 4: /Main IC1/D3#_SCL -> /Main IC1/D11#
- SW38 pad 1: /Main IC1/D4 -> /Right Switch Matrix/COL_0_R
- SW46 pad 1: /Main IC1/D4 -> /Right Switch Matrix/COL_0_R
- SW53 pad 1: /Right Switch Matrix/RE_SW1 -> /Right Switch Matrix/COL_7_R
- SW54 pad 1: /Main IC1/D4 -> /Right Switch Matrix/COL_0_R
- SW62 pad 1: /Main IC1/D4 -> /Right Switch Matrix/COL_0_R
- SW70 pad 1: /Main IC1/D4 -> /Right Switch Matrix/COL_0_R
- SW78 pad 1: /Right Switch Matrix/COL_1_R -> /Right Switch Matrix/COL_0_R
- SW79 pad 1: /Right Switch Matrix/COL_2_R -> /Right Switch Matrix/COL_1_R
- SW80 pad 1: /Right Switch Matrix/COL_3_R -> /Right Switch Matrix/COL_2_R
- SW81 pad 1: /Right Switch Matrix/COL_4_R -> /Right Switch Matrix/COL_3_R
- SW82 pad 1: /Right Switch Matrix/COL_5_R -> /Right Switch Matrix/COL_4_R
- SW83 pad 1: /Right Switch Matrix/COL_6_R -> /Right Switch Matrix/COL_5_R
- SW84 pad 1: /Right Switch Matrix/COL_7_R -> /Right Switch Matrix/COL_6_R
- U9 pad 1: /Main IC1/D7 -> /~{Q7}
- U9 pad 25: /Main IC1/D4 -> /CP
- U9 pad 26: /Main IC1/D12 -> /RE_1_A
- U9 pad 27: /Main IC1/D6# -> /~{PL}
- U9 pad 28: /Main IC1/D8 -> /DS
- U9 pad 29: /Main IC1/D9# -> /ST_CP
- U9 pad 30: /Main IC1/D10# -> /SH_CP
- U9 pad 31: /Main IC1/D5# -> /~{CE}
- U9 pad 32: /Main IC1/D13# -> /RE_1_B
- U9 pad 36: /Main IC1/A0 -> /RE_SW
Routing:
- net +5V: track 0.00 -> 1475.4 mm, vias 0 -> 6
- net GND: track 0.00 -> 1118.2 mm, vias 0 -> 5
- net /Right Switch Matrix/COL_7_R: track 0.00 -> 299.2 mm
- net /Right Switch Matrix/ROW_0_R: track 0.00 -> 277.7 mm, vias 0 -> 1
- net /Right Switch Matrix/ROW_1_R: track 0.00 -> 276.0 mm, vias 0 -> 1
- net /Right Switch Matrix/ROW_3_R: track 0.00 -> 267.5 mm, vias 0 -> 1
- net /Right Switch Matrix/COL_6_R: track 0.00 -> 264.8 mm
- net /Right Switch Matrix/COL_5_R: track 0.00 -> 231.1 mm
- net /Right Switch Matrix/ROW_2_R: track 0.00 -> 220.6 mm, vias 0 -> 1
- net /Right Switch Matrix/ROW_5_R: track 0.00 -> 213.4 mm, vias 0 -> 1
- net /Right Switch Matrix/COL_4_R: track 0.00 -> 210.6 mm
- net /Right Switch Matrix/ROW_4_R: track 0.00 -> 204.9 mm, vias 0 -> 1
- net /Right Switch Matrix/COL_3_R: track 0.00 -> 199.7 mm
- net /RE_1_A: track 0.00 -> 195.4 mm
- net /RE_1_B: track 0.00 -> 183.4 mm
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Other:
- board outline added: 181 x 114.3 mm

Commit message: better silkscreen
Parts:
- removed C102, C103, C104, C105, C106, C107, C108, C109, C110, C111, C112, C113, C114, C115, C116, C117, C118, C119, C120, C121, C16, C17, C18, C19, C20, C21, C214, C22, C23, C24, C25, C26, C27, C28, C29, C30, C31, C32, C33, C34, C35, C36, C37, C38, C39, C40, C41, C42, C43, C44, C45, C46, C47, C48, C49, C50, C51: 100n, Capacitor_SMD:C_0603_1608Metric
- removed C122, C123, C124, C125, C126, C127, C128, C129: 10n, Capacitor_SMD:C_0603_1608Metric
- removed C211, C213: 22u, Capacitor_SMD:C_0603_1608Metric
- removed C212: 10u, Capacitor_SMD:C_0603_1608Metric
- removed D10, D100, D101, D102, D103, D104, D105, D106, D107, D108, D109, D11, D110, D111, D112, D113, D114, D12, D13, D14, D15, D16, D17, D18, D19, D20, D21, D22, D23, D24, D25, D26, D27, D28, D29, D30, D31, D32, D33, D34, D35, D36, D37, D38, D39, D40, D41, D42, D7, D8, D9, D91, D92, D93, D94, D95, D96, D97, D98, D99: 1N4148W, Diode_SMD:D_SOD-123
- removed D127: SS34, Diode_SMD:D_SMC
- removed D128: Red, LED_SMD:LED_0805_2012Metric
- removed D129: Green, LED_SMD:LED_0805_2012Metric
- removed L1: 22uH, Inductor_SMD:L_7.3x7.3_H4.5
- removed Q1, Q2, Q3: FDN340P, Package_TO_SOT_SMD:SOT-23
- removed Q4: FS8205, Package_TO_SOT_SMD:SOT-23-6
- removed R1, R51, R63, R79, R84, R90, R91, R97: 1M, Resistor_SMD:R_0603_1608Metric
- removed R103: 7.5K, Resistor_SMD:R_0603_1608Metric
- removed R104, R105, R106, R107, R108, R110, R111: 1k, Resistor_SMD:R_0603_1608Metric
- removed R31, R32, R33, R34, R35, R36, R37, R38, R39, R40, R41, R42, R43, R44, R45, R46, R47, R48, R49, R50: 10K, Resistor_SMD:R_0603_1608Metric
- removed RE2, RE3, RE4, RE5: EC11, Rotary_Encoder:RotaryEncoder_Alps_EC11E-Switch_Vertical_H20mm
- removed RGB1, RGB10, RGB100, RGB101, RGB102, RGB103, RGB104, RGB11, RGB12, RGB13, RGB14, RGB15, RGB16, RGB17, RGB18, RGB19, RGB2, RGB20, RGB21, RGB22, RGB23, RGB24, RGB25, RGB26, RGB27, RGB28, RGB29, RGB3, RGB30, RGB31, RGB32, RGB33, RGB34, RGB35, RGB36, RGB4, RGB5, RGB6, RGB7, RGB8, RGB85, RGB86, RGB87, RGB88, RGB89, RGB9, RGB90, RGB91, RGB92, RGB93, RGB94, RGB95, RGB96, RGB97, RGB98, RGB99: WS2812B, LED_SMD:LED_WS2812B_PLCC4_5.0x5.0mm_P3.2mm
- removed SW10: 1, Button_Switch_Keyboard:SW_Cherry_MX_1.00u_PCB
- removed SW100: NUMPAD15, Button_Switch_Keyboard:SW_Cherry_MX_1.00u_PCB
- removed SW101: NUMPAD16, Button_Switch_Keyboard:SW_Cherry_MX_1.00u_PCB
- removed SW102: NUMPAD17, Button_Switch_Keyboard:SW_Cherry_MX_1.00u_PCB
- removed SW103: NUMPAD18, Button_Switch_Keyboard:SW_Cherry_MX_1.00u_PCB
- removed SW104: NUMPAD19, Button_Switch_Keyboard:SW_Cherry_MX_1.00u_PCB
- removed SW105: NUMPAD20, Button_Switch_Keyboard:SW_Cherry_MX_1.00u_PCB
- removed SW108: Battery Switch, Connector_PinHeader_2.54mm:PinHeader_1x03_P2.54mm_Vertical
- removed SW11: 2, Button_Switch_Keyboard:SW_Cherry_MX_1.00u_PCB
- removed SW12: 3, Button_Switch_Keyboard:SW_Cherry_MX_1.00u_PCB
- removed SW13: 4, Button_Switch_Keyboard:SW_Cherry_MX_1.00u_PCB
- removed SW14: 5, Button_Switch_Keyboard:SW_Cherry_MX_1.00u_PCB
- removed SW15: 6, Button_Switch_Keyboard:SW_Cherry_MX_1.00u_PCB
- removed SW16: TAB, Button_Switch_Keyboard:SW_Cherry_MX_1.50u_PCB
- removed SW17: Q, Button_Switch_Keyboard:SW_Cherry_MX_1.00u_PCB
- removed SW18: W, Button_Switch_Keyboard:SW_Cherry_MX_1.00u_PCB
- removed SW19: E, Button_Switch_Keyboard:SW_Cherry_MX_1.00u_PCB
- removed SW2: ESC, Button_Switch_Keyboard:SW_Cherry_MX_1.00u_PCB
- removed SW20: R, Button_Switch_Keyboard:SW_Cherry_MX_1.00u_PCB
- removed SW21: T, Button_Switch_Keyboard:SW_Cherry_MX_1.00u_PCB
- removed SW22: MAYUS, Button_Switch_Keyboard:SW_Cherry_MX_1.75u_PCB
- removed SW23: A, Button_Switch_Keyboard:SW_Cherry_MX_1.00u_PCB
- removed SW24: S, Button_Switch_Keyboard:SW_Cherry_MX_1.00u_PCB
- removed SW25: D, Button_Switch_Keyboard:SW_Cherry_MX_1.00u_PCB
- removed SW26: F, Button_Switch_Keyboard:SW_Cherry_MX_1.00u_PCB
- removed SW27: G, Button_Switch_Keyboard:SW_Cherry_MX_1.00u_PCB
- removed SW28: L_SHIFT, Button_Switch_Keyboard:SW_Cherry_MX_2.25u_PCB
- removed SW29: Z, Button_Switch_Keyboard:SW_Cherry_MX_1.00u_PCB
- removed SW3: F1, Button_Switch_Keyboard:SW_Cherry_MX_1.00u_PCB
- removed SW30: X, Button_Switch_Keyboard:SW_Cherry_MX_1.00u_PCB
- removed SW31: C, Button_Switch_Keyboard:SW_Cherry_MX_1.00u_PCB
- removed SW32: V, Button_Switch_Keyboard:SW_Cherry_MX_1.00u_PCB
- removed SW33: B, Button_Switch_Keyboard:SW_Cherry_MX_1.00u_PCB
- removed SW34: L_CRTL, Button_Switch_Keyboard:SW_Cherry_MX_1.25u_PCB
- removed SW35: OS, Button_Switch_Keyboard:SW_Cherry_MX_1.25u_PCB
- removed SW36: L_ALT, Button_Switch_Keyboard:SW_Cherry_MX_1.25u_PCB
- removed SW37: L_SPACE, Button_Switch_Keyboard:SW_Cherry_MX_2.75u_PCB
- removed SW4: F2, Button_Switch_Keyboard:SW_Cherry_MX_1.00u_PCB
- removed SW5: F3, Button_Switch_Keyboard:SW_Cherry_MX_1.00u_PCB
- removed SW6: F4, Button_Switch_Keyboard:SW_Cherry_MX_1.00u_PCB
- removed SW7: F5, Button_Switch_Keyboard:SW_Cherry_MX_1.00u_PCB
- removed SW8: F6, Button_Switch_Keyboard:SW_Cherry_MX_1.00u_PCB
- removed SW86: NUMPAD1, Button_Switch_Keyboard:SW_Cherry_MX_1.00u_PCB
- removed SW87: NUMPAD2, Button_Switch_Keyboard:SW_Cherry_MX_1.00u_PCB
- removed SW88: NUMPAD3, Button_Switch_Keyboard:SW_Cherry_MX_1.00u_PCB
- removed SW89: NUMPAD4, Button_Switch_Keyboard:SW_Cherry_MX_1.00u_PCB
- removed SW9: `, Button_Switch_Keyboard:SW_Cherry_MX_1.00u_PCB
- removed SW90: NUMPAD5, Button_Switch_Keyboard:SW_Cherry_MX_1.00u_PCB
- removed SW91: NUMPAD6, Button_Switch_Keyboard:SW_Cherry_MX_1.00u_PCB
- removed SW92: NUMPAD7, Button_Switch_Keyboard:SW_Cherry_MX_1.00u_PCB
- removed SW93: NUMPAD8, Button_Switch_Keyboard:SW_Cherry_MX_1.00u_PCB
- removed SW94: NUMPAD9, Button_Switch_Keyboard:SW_Cherry_MX_1.00u_PCB
- removed SW95: NUMPAD10, Button_Switch_Keyboard:SW_Cherry_MX_1.00u_PCB
- removed SW96: NUMPAD11, Button_Switch_Keyboard:SW_Cherry_MX_1.00u_PCB
- removed SW97: NUMPAD12, Button_Switch_Keyboard:SW_Cherry_MX_1.00u_PCB
- removed SW98: NUMPAD13, Button_Switch_Keyboard:SW_Cherry_MX_1.00u_PCB
- removed SW99: NUMPAD14, Button_Switch_Keyboard:SW_Cherry_MX_1.00u_PCB
- removed U11, U15, U5: LP2985-33DBVR, Package_TO_SOT_SMD:SOT-23-5
- removed U12, U2, U8: NCP1117ST50T3G, Package_TO_SOT_SMD:SOT-223-3_TabPin2
- removed U13, U3, U9: ATmega32U4, Package_QFP:TQFP-44_10x10mm_P0.8mm
- removed U17, U20: TPS2561, Package_SON:VSON-10-1EP_3x3mm_P0.5mm_EP1.65x2.4mm_ThermalVias
- removed U18, U21: TLV71311PDBVR, Package_TO_SOT_SMD:TSOT-23-5
- removed U19, U23: TLV70033DDCR, Package_TO_SOT_SMD:TSOT-23-5
- removed U21: TP4056, Package_SO:SOP-8-1EP_4.57x4.57mm_P1.27mm_EP4.57x4.45mm_ThermalVias
- removed U22: MT3608, Package_TO_SOT_SMD:SOT-23-6
- removed U23: FS312F-G, Package_TO_SOT_SMD:SOT-23-6
- moved C100 154.1 mm to (334.6, 136.4)
- moved C101 154.1 mm to (328.3, 136.4)
- moved C59 154.1 mm to (211.6, 132.2)
- moved C62 154.1 mm to (283.8, 168.4)
- moved C63 154.1 mm to (331.4, 225.6)
- moved C64 154.1 mm to (236.1, 225.6)
- moved C66 154.1 mm to (177.6, 172.6)
- moved C70 154.1 mm to (331.4, 206.5)
- moved C71 154.1 mm to (308.8, 206.5)
- moved C72 154.1 mm to (221.8, 206.5)
- moved C74 154.1 mm to (331.4, 187.5)
- moved C76 154.1 mm to (249.7, 132.2)
- moved C78 154.1 mm to (268.8, 132.2)
- moved C81 154.1 mm to (284.6, 206.5)
- moved C84 154.1 mm to (300.4, 187.5)
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Routing:
- net GND: track 1118.2 -> 1409.2 mm, vias 5 -> 26
- net +5V: track 1475.4 -> 1485.3 mm, vias 6 -> 7
- net /Right Switch Matrix/ROW_5_R: track 213.4 -> 214.3 mm
Other:
- outline, holes or cut-outs redrawn

Commit message: Started USB hub layout and added footprints
Parts:
- added C102: 100n, Capacitor_SMD:C_0603_1608Metric, F.Cu at (70.4, 69.7)
- added C103: 100n, Capacitor_SMD:C_0603_1608Metric, F.Cu at (70.4, 72.2)
- added C104: 100n, Capacitor_SMD:C_0603_1608Metric, F.Cu at (70.4, 74.7)
- added C105: 100n, Capacitor_SMD:C_0603_1608Metric, F.Cu at (70.4, 77.2)
- added C106: 100n, Capacitor_SMD:C_0603_1608Metric, F.Cu at (70.4, 79.7)
- added C107: 100n, Capacitor_SMD:C_0603_1608Metric, F.Cu at (70.4, 82.2)
- added C108: 100n, Capacitor_SMD:C_0603_1608Metric, F.Cu at (70.4, 84.7)
- added C109: 100n, Capacitor_SMD:C_0603_1608Metric, F.Cu at (70.4, 87.2)
- added C110: 100n, Capacitor_SMD:C_0603_1608Metric, F.Cu at (74.5, 69.7)
- added C111: 100n, Capacitor_SMD:C_0603_1608Metric, F.Cu at (74.5, 72.2)
- added C112: 100n, Capacitor_SMD:C_0603_1608Metric, F.Cu at (74.5, 74.7)
- added C113: 100n, Capacitor_SMD:C_0603_1608Metric, F.Cu at (74.5, 77.2)
- added C114: 100n, Capacitor_SMD:C_0603_1608Metric, F.Cu at (74.5, 79.7)
- added C115: 100n, Capacitor_SMD:C_0603_1608Metric, F.Cu at (74.5, 82.2)
- added C116: 100n, Capacitor_SMD:C_0603_1608Metric, F.Cu at (74.5, 84.7)
- added C117: 100n, Capacitor_SMD:C_0603_1608Metric, F.Cu at (74.5, 87.2)
- added C118: 100n, Capacitor_SMD:C_0603_1608Metric, F.Cu at (78.5, 69.7)
- added C119: 100n, Capacitor_SMD:C_0603_1608Metric, F.Cu at (78.5, 72.2)
- added C120: 100n, Capacitor_SMD:C_0603_1608Metric, F.Cu at (78.5, 74.7)
- added C121: 100n, Capacitor_SMD:C_0603_1608Metric, F.Cu at (78.5, 77.2)
- added C122: 10n, Capacitor_SMD:C_0603_1608Metric, F.Cu at (78.5, 79.7)
- added C123: 10n, Capacitor_SMD:C_0603_1608Metric, F.Cu at (78.5, 82.2)
- added C124: 10n, Capacitor_SMD:C_0603_1608Metric, F.Cu at (78.5, 84.7)
- added C125: 10n, Capacitor_SMD:C_0603_1608Metric, F.Cu at (78.5, 87.2)
- added C126: 10n, Capacitor_SMD:C_0603_1608Metric, F.Cu at (82.5, 69.7)
- added C127: 10n, Capacitor_SMD:C_0603_1608Metric, F.Cu at (82.5, 72.2)
- added C128: 10n, Capacitor_SMD:C_0603_1608Metric, F.Cu at (82.5, 74.7)
- added C129: 10n, Capacitor_SMD:C_0603_1608Metric, F.Cu at (82.5, 77.2)
- added C16: 100n, Capacitor_SMD:C_0603_1608Metric, F.Cu at (162.7, -85.3)
- added C160: 1n, Capacitor_SMD:C_0603_1608Metric, F.Cu at (220.1, 62.4)
- added C161: 100n, Capacitor_SMD:C_0603_1608Metric, F.Cu at (220.1, 64.9)
- added C163: 100n, Capacitor_SMD:C_0603_1608Metric, F.Cu at (220.1, 67.4)
- added C164: 100n, Capacitor_SMD:C_0603_1608Metric, F.Cu at (220.1, 69.9)
- added C165: 20p, Capacitor_SMD:C_0603_1608Metric, F.Cu at (220.1, 72.5)
- added C166: 20p, Capacitor_SMD:C_0603_1608Metric, F.Cu at (220.1, 75.0)
- added C167: 1u, Capacitor_SMD:C_0603_1608Metric, F.Cu at (223.4, 111.8)
- added C168: 1n, Capacitor_SMD:C_0603_1608Metric, F.Cu at (220.1, 77.5)
- added C169: 1n, Capacitor_SMD:C_0603_1608Metric, F.Cu at (220.1, 80.0)
- added C17: 100n, Capacitor_SMD:C_0603_1608Metric, F.Cu at (162.7, -82.8)
- added C170: 100n, Capacitor_SMD:C_0603_1608Metric, F.Cu at (220.1, 82.5)
- added C171: 100n, Capacitor_SMD:C_0603_1608Metric, F.Cu at (220.1, 85.0)
- added C172: 100n, Capacitor_SMD:C_0603_1608Metric, F.Cu at (220.1, 87.5)
- added C173: 100n, Capacitor_SMD:C_0603_1608Metric, F.Cu at (220.1, 90.0)
- added C174: 100n, Capacitor_SMD:C_0603_1608Metric, F.Cu at (224.1, 62.4)
- added C175: 100n, Capacitor_SMD:C_0603_1608Metric, F.Cu at (224.1, 64.9)
- added C176: 10u, Capacitor_Tantalum_SMD:CP_EIA-3216-18_Kemet-A, F.Cu at (245.1, 62.7)
- added C177: 100n, Capacitor_SMD:C_0603_1608Metric, F.Cu at (224.1, 67.4)
- added C178: 100n, Capacitor_SMD:C_0603_1608Metric, F.Cu at (224.1, 69.9)
- added C179: 100n, Capacitor_SMD:C_0603_1608Metric, F.Cu at (224.1, 72.5)
- added C18: 100n, Capacitor_SMD:C_0603_1608Metric, F.Cu at (162.7, -80.3)
- added C180: 100n, Capacitor_SMD:C_0603_1608Metric, F.Cu at (224.1, 75.0)
- added C181: 100n, Capacitor_SMD:C_0603_1608Metric, F.Cu at (224.1, 77.5)
- added C182: 100n, Capacitor_SMD:C_0603_1608Metric, F.Cu at (224.1, 80.0)
- added C183: 100n, Capacitor_SMD:C_0603_1608Metric, F.Cu at (224.1, 82.5)
- added C184: 100n, Capacitor_SMD:C_0603_1608Metric, F.Cu at (224.1, 85.0)
- added C185: 100n, Capacitor_SMD:C_0603_1608Metric, F.Cu at (224.1, 87.5)
- added C186: 100n, Capacitor_SMD:C_0603_1608Metric, F.Cu at (224.1, 90.0)
- added C187: 100n, Capacitor_SMD:C_0603_1608Metric, F.Cu at (228.2, 62.4)
- added C188: 100n, Capacitor_SMD:C_0603_1608Metric, F.Cu at (228.2, 64.9)
- added C189: 10u, Capacitor_Tantalum_SMD:CP_EIA-3216-18_Kemet-A, F.Cu at (245.1, 65.9)
- added C19: 100n, Capacitor_SMD:C_0603_1608Metric, F.Cu at (162.7, -77.8)
- added C190: 100n, Capacitor_SMD:C_0603_1608Metric, F.Cu at (228.2, 67.4)
- added C191: 100n, Capacitor_SMD:C_0603_1608Metric, F.Cu at (228.2, 69.9)
- added C192: 1n, Capacitor_SMD:C_0603_1608Metric, F.Cu at (228.2, 72.5)
- added C193: 100n, Capacitor_SMD:C_0603_1608Metric, F.Cu at (228.2, 75.0)
- added C194: 100n, Capacitor_SMD:C_0603_1608Metric, F.Cu at (228.2, 77.5)
- added C195: 1u X5R, Capacitor_SMD:C_0603_1608Metric, F.Cu at (228.2, 80.0)
- added C196: 1u X5R, Capacitor_SMD:C_0603_1608Metric, F.Cu at (228.2, 82.5)
- added C197: 150u, Capacitor_Tantalum_SMD:CP_EIA-3216-18_Kemet-A, F.Cu at (245.1, 69.0)
- added C198: 100n, Capacitor_SMD:C_0603_1608Metric, F.Cu at (228.2, 85.0)
- added C199: 150u, Capacitor_Tantalum_SMD:CP_EIA-3216-18_Kemet-A, F.Cu at (245.1, 72.2)
- added C20: 100n, Capacitor_SMD:C_0603_1608Metric, F.Cu at (162.7, -75.3)
- added C200: 100n, Capacitor_SMD:C_0603_1608Metric, F.Cu at (228.2, 87.5)
- added C201: 100n, Capacitor_SMD:C_0603_1608Metric, F.Cu at (228.2, 90.0)
- added C202: 1u X5R, Capacitor_SMD:C_0603_1608Metric, F.Cu at (232.2, 62.4)
- added C203: 1u X5R, Capacitor_SMD:C_0603_1608Metric, F.Cu at (232.2, 64.9)
- added C204: 100n, Capacitor_SMD:C_0603_1608Metric, F.Cu at (232.2, 67.4)
- added C205: 100n, Capacitor_SMD:C_0603_1608Metric, F.Cu at (232.2, 69.9)
- added C206: 100n, Capacitor_SMD:C_0603_1608Metric, F.Cu at (232.2, 72.5)
- added C207: 150u, Capacitor_Tantalum_SMD:CP_EIA-3216-18_Kemet-A, F.Cu at (245.1, 75.3)
- added C208: 100n, Capacitor_SMD:C_0603_1608Metric, F.Cu at (232.2, 75.0)
- added C209: 150u, Capacitor_Tantalum_SMD:CP_EIA-3216-18_Kemet-A, F.Cu at (245.1, 78.5)
- added C21: 100n, Capacitor_SMD:C_0603_1608Metric, F.Cu at (162.7, -72.8)
- added C210: 100n, Capacitor_SMD:C_0603_1608Metric, F.Cu at (232.2, 77.5)
- added C211: 22u, Capacitor_SMD:C_0603_1608Metric, F.Cu at (163.5, 42.5)
- added C212: 10u, Capacitor_SMD:C_0603_1608Metric, F.Cu at (163.5, 45.0)
- added C213: 22u, Capacitor_SMD:C_0603_1608Metric, F.Cu at (163.5, 47.5)
- added C214: 100n, Capacitor_SMD:C_0603_1608Metric, F.Cu at (163.5, 50.0)
- added C22: 100n, Capacitor_SMD:C_0603_1608Metric, F.Cu at (162.7, -70.3)
- added C23: 100n, Capacitor_SMD:C_0603_1608Metric, F.Cu at (162.7, -67.7)
- added C24: 100n, Capacitor_SMD:C_0603_1608Metric, F.Cu at (162.7, -65.2)
- added C25: 100n, Capacitor_SMD:C_0603_1608Metric, F.Cu at (166.7, -85.3)
- added C26: 100n, Capacitor_SMD:C_0603_1608Metric, F.Cu at (166.7, -82.8)
- added C27: 100n, Capacitor_SMD:C_0603_1608Metric, F.Cu at (166.7, -80.3)
- added C28: 100n, Capacitor_SMD:C_0603_1608Metric, F.Cu at (166.7, -77.8)
- added C29: 100n, Capacitor_SMD:C_0603_1608Metric, F.Cu at (166.7, -75.3)
- added C30: 100n, Capacitor_SMD:C_0603_1608Metric, F.Cu at (166.7, -72.8)
- added C31: 100n, Capacitor_SMD:C_0603_1608Metric, F.Cu at (166.7, -70.3)
- added C32: 100n, Capacitor_SMD:C_0603_1608Metric, F.Cu at (166.7, -67.7)
- added C33: 100n, Capacitor_SMD:C_0603_1608Metric, F.Cu at (166.7, -65.2)
- added C34: 100n, Capacitor_SMD:C_0603_1608Metric, F.Cu at (170.7, -85.3)
- added C35: 100n, Capacitor_SMD:C_0603_1608Metric, F.Cu at (170.7, -82.8)
- added C36: 100n, Capacitor_SMD:C_0603_1608Metric, F.Cu at (170.7, -80.3)
- added C37: 100n, Capacitor_SMD:C_0603_1608Metric, F.Cu at (170.7, -77.8)
- added C38: 100n, Capacitor_SMD:C_0603_1608Metric, F.Cu at (170.7, -75.3)
- added C39: 100n, Capacitor_SMD:C_0603_1608Metric, F.Cu at (170.7, -72.8)
- added C40: 100n, Capacitor_SMD:C_0603_1608Metric, F.Cu at (170.7, -70.3)
- added C41: 100n, Capacitor_SMD:C_0603_1608Metric, F.Cu at (170.7, -67.7)
- added C42: 100n, Capacitor_SMD:C_0603_1608Metric, F.Cu at (170.7, -65.2)
- added C43: 100n, Capacitor_SMD:C_0603_1608Metric, F.Cu at (174.8, -85.3)
- added C44: 100n, Capacitor_SMD:C_0603_1608Metric, F.Cu at (174.8, -82.8)
- added C45: 100n, Capacitor_SMD:C_0603_1608Metric, F.Cu at (174.8, -80.3)
- added C46: 100n, Capacitor_SMD:C_0603_1608Metric, F.Cu at (174.8, -77.8)
- added C47: 100n, Capacitor_SMD:C_0603_1608Metric, F.Cu at (174.8, -75.3)
- added C48: 100n, Capacitor_SMD:C_0603_1608Metric, F.Cu at (174.8, -72.8)
- added C49: 100n, Capacitor_SMD:C_0603_1608Metric, F.Cu at (174.8, -70.3)
- added C50: 100n, Capacitor_SMD:C_0603_1608Metric, F.Cu at (174.8, -67.7)
- added C51: 100n, Capacitor_SMD:C_0603_1608Metric, F.Cu at (174.8, -65.2)
- added D10: 1N4148W, Diode_SMD:D_SOD-123, F.Cu at (163.6, -105.0)
- added D100: 1N4148W, Diode_SMD:D_SOD-123, F.Cu at (101.2, 80.1)
- added D101: 1N4148W, Diode_SMD:D_SOD-123, F.Cu at (101.2, 83.5)
- added D102: 1N4148W, Diode_SMD:D_SOD-123, F.Cu at (101.2, 86.8)
- added D103: 1N4148W, Diode_SMD:D_SOD-123, F.Cu at (107.0, 70.1)
- added D104: 1N4148W, Diode_SMD:D_SOD-123, F.Cu at (107.0, 73.4)
- added D105: 1N4148W, Diode_SMD:D_SOD-123, F.Cu at (107.0, 76.8)
- added D106: 1N4148W, Diode_SMD:D_SOD-123, F.Cu at (107.0, 80.1)
- added D107: 1N4148W, Diode_SMD:D_SOD-123, F.Cu at (107.0, 83.5)
- added D108: 1N4148W, Diode_SMD:D_SOD-123, F.Cu at (107.0, 86.8)
- added D109: 1N4148W, Diode_SMD:D_SOD-123, F.Cu at (112.8, 70.1)
- added D11: 1N4148W, Diode_SMD:D_SOD-123, F.Cu at (163.6, -101.6)
- added D110: 1N4148W, Diode_SMD:D_SOD-123, F.Cu at (112.8, 73.4)
- added D111: 1N4148W, Diode_SMD:D_SOD-123, F.Cu at (112.8, 76.8)
- added D112: 1N4148W, Diode_SMD:D_SOD-123, F.Cu at (112.8, 80.1)
- added D113: 1N4148W, Diode_SMD:D_SOD-123, F.Cu at (112.8, 83.5)
- added D114: 1N4148W, Diode_SMD:D_SOD-123, F.Cu at (112.8, 86.8)
- added D12: 1N4148W, Diode_SMD:D_SOD-123, F.Cu at (163.6, -98.3)
- added D127: SS34, Diode_SMD:D_SMC, F.Cu at (166.9, 55.2)
- added D128: Red, LED_SMD:LED_0805_2012Metric, F.Cu at (180.4, 42.8)
- added D129: Green, LED_SMD:LED_0805_2012Metric, F.Cu at (180.4, 45.8)
- added D13: 1N4148W, Diode_SMD:D_SOD-123, F.Cu at (163.6, -94.9)
- added D14: 1N4148W, Diode_SMD:D_SOD-123, F.Cu at (163.6, -91.6)
- added D15: 1N4148W, Diode_SMD:D_SOD-123, F.Cu at (163.6, -88.2)
- added D16: 1N4148W, Diode_SMD:D_SOD-123, F.Cu at (169.4, -115.0)
- added D17: 1N4148W, Diode_SMD:D_SOD-123, F.Cu at (169.4, -111.7)
- added D18: 1N4148W, Diode_SMD:D_SOD-123, F.Cu at (169.4, -108.3)
- added D19: 1N4148W, Diode_SMD:D_SOD-123, F.Cu at (169.4, -105.0)
- added D20: 1N4148W, Diode_SMD:D_SOD-123, F.Cu at (169.4, -101.6)
- added D21: 1N4148W, Diode_SMD:D_SOD-123, F.Cu at (169.4, -98.3)
- added D22: 1N4148W, Diode_SMD:D_SOD-123, F.Cu at (169.4, -94.9)
- added D23: 1N4148W, Diode_SMD:D_SOD-123, F.Cu at (169.4, -91.6)
- added D24: 1N4148W, Diode_SMD:D_SOD-123, F.Cu at (169.4, -88.2)
- added D25: 1N4148W, Diode_SMD:D_SOD-123, F.Cu at (175.2, -115.0)
- added D26: 1N4148W, Diode_SMD:D_SOD-123, F.Cu at (175.2, -111.7)
- added D27: 1N4148W, Diode_SMD:D_SOD-123, F.Cu at (175.2, -108.3)
- added D28: 1N4148W, Diode_SMD:D_SOD-123, F.Cu at (175.2, -105.0)
- added D29: 1N4148W, Diode_SMD:D_SOD-123, F.Cu at (175.2, -101.6)
- added D30: 1N4148W, Diode_SMD:D_SOD-123, F.Cu at (175.2, -98.3)
- added D31: 1N4148W, Diode_SMD:D_SOD-123, F.Cu at (175.2, -94.9)
- added D32: 1N4148W, Diode_SMD:D_SOD-123, F.Cu at (175.2, -91.6)
- added D33: 1N4148W, Diode_SMD:D_SOD-123, F.Cu at (175.2, -88.2)
- added D34: 1N4148W, Diode_SMD:D_SOD-123, F.Cu at (181.0, -115.0)
- added D35: 1N4148W, Diode_SMD:D_SOD-123, F.Cu at (181.0, -111.7)
- added D36: 1N4148W, Diode_SMD:D_SOD-123, F.Cu at (181.0, -108.3)
- added D37: 1N4148W, Diode_SMD:D_SOD-123, F.Cu at (181.0, -105.0)
- added D38: 1N4148W, Diode_SMD:D_SOD-123, F.Cu at (181.0, -101.6)
- added D39: 1N4148W, Diode_SMD:D_SOD-123, F.Cu at (181.0, -98.3)
- added D40: 1N4148W, Diode_SMD:D_SOD-123, F.Cu at (181.0, -94.9)
- added D41: 1N4148W, Diode_SMD:D_SOD-123, F.Cu at (181.0, -91.6)
- added D42: 1N4148W, Diode_SMD:D_SOD-123, F.Cu at (181.0, -88.2)
- added D7: 1N4148W, Diode_SMD:D_SOD-123, F.Cu at (163.6, -115.0)
- added D8: 1N4148W, Diode_SMD:D_SOD-123, F.Cu at (163.6, -111.7)
- added D9: 1N4148W, Diode_SMD:D_SOD-123, F.Cu at (163.6, -108.3)
- added D91: 1N4148W, Diode_SMD:D_SOD-123, F.Cu at (95.4, 70.1)
- added D92: 1N4148W, Diode_SMD:D_SOD-123, F.Cu at (95.4, 73.4)
- added D93: 1N4148W, Diode_SMD:D_SOD-123, F.Cu at (95.4, 76.8)
- added D94: 1N4148W, Diode_SMD:D_SOD-123, F.Cu at (95.4, 80.1)
- added D95: 1N4148W, Diode_SMD:D_SOD-123, F.Cu at (95.4, 83.5)
- added D96: 1N4148W, Diode_SMD:D_SOD-123, F.Cu at (95.4, 86.8)
- added D97: 1N4148W, Diode_SMD:D_SOD-123, F.Cu at (101.2, 70.1)
- added D98: 1N4148W, Diode_SMD:D_SOD-123, F.Cu at (101.2, 73.4)
- added D99: 1N4148W, Diode_SMD:D_SOD-123, F.Cu at (101.2, 76.8)
- added FB10: >50mΩ 220Ω @ 100MHz, Inductor_SMD:L_0805_2012Metric, F.Cu at (250.2, 70.8)
- added FB11: >50mΩ 220Ω @ 100MHz, Inductor_SMD:L_0805_2012Metric, F.Cu at (250.2, 73.5)
- added FB12: >50mΩ 220Ω @ 100MHz, Inductor_SMD:L_0805_2012Metric, F.Cu at (250.2, 76.3)
- added FB7: >50mΩ 220Ω @ 100MHz, Inductor_SMD:L_0805_2012Metric, F.Cu at (250.2, 62.5)
- added FB8: >50mΩ 220Ω @ 100MHz, Inductor_SMD:L_0805_2012Metric, F.Cu at (250.2, 65.3)
- added FB9: >50mΩ 220Ω @ 100MHz, Inductor_SMD:L_0805_2012Metric, F.Cu at (250.2, 68.0)
- added J6: UPSTREAM, Connector_USB:USB_C_Receptacle_Amphenol_12401610E4-2A, F.Cu at (217.2, 100.3)
- added J7: DOWNSTREAM_3, Connector_USB:USB3_A_Molex_48393-001, F.Cu at (267.0, 105.0)
- added J8: DOWNSTREAM_1, Connector_USB:USB_C_Receptacle_Amphenol_12401610E4-2A, F.Cu at (248.2, 100.3)
- added J9: DOWNSTREAM_2, Connector_USB:USB_C_Receptacle_Amphenol_12401610E4-2A, F.Cu at (278.7, 100.3)
- added L1: 22uH, Inductor_SMD:L_7.3x7.3_H4.5, F.Cu at (178.2, 55.4)
- added Q1: FDN340P, Package_TO_SOT_SMD:SOT-23, F.Cu at (173.2, 64.0)
- added Q2: FDN340P, Package_TO_SOT_SMD:SOT-23, F.Cu at (194.5, 64.0)
- added Q3: FDN340P, Package_TO_SOT_SMD:SOT-23, F.Cu at (201.8, 37.3)
- added Q4: FS8205, Package_TO_SOT_SMD:SOT-23-6, F.Cu at (158.9, 37.3)
- added R1: 1M, Resistor_SMD:R_0603_1608Metric, F.Cu at (172.8, 67.5)
- added R100: 10k, Resistor_SMD:R_0603_1608Metric, F.Cu at (240.2, 82.5)
- added R101: 5.1k, Resistor_SMD:R_0603_1608Metric, F.Cu at (240.2, 85.0)
- added R102: 25.5k, Resistor_SMD:R_0603_1608Metric, F.Cu at (240.2, 87.5)
- added R103: 7.5K, Resistor_SMD:R_0603_1608Metric, F.Cu at (167.5, 42.5)
- added R104: 1k, Resistor_SMD:R_0603_1608Metric, F.Cu at (167.5, 45.0)
- added R105: 1k, Resistor_SMD:R_0603_1608Metric, F.Cu at (167.5, 47.5)
- added R106: 1k, Resistor_SMD:R_0603_1608Metric, F.Cu at (167.5, 50.0)
- added R107: 1k, Resistor_SMD:R_0603_1608Metric, F.Cu at (171.5, 42.5)
- added R108: 1k, Resistor_SMD:R_0603_1608Metric, F.Cu at (171.5, 45.0)
- added R110: 1k, Resistor_SMD:R_0603_1608Metric, F.Cu at (171.5, 47.5)
- added R111: 1k, Resistor_SMD:R_0603_1608Metric, F.Cu at (171.5, 50.0)
- added R31: 10K, Resistor_SMD:R_0603_1608Metric, F.Cu at (82.5, 79.7)
- added R32: 10K, Resistor_SMD:R_0603_1608Metric, F.Cu at (82.5, 82.2)
- added R33: 10K, Resistor_SMD:R_0603_1608Metric, F.Cu at (82.5, 84.7)
- added R34: 10K, Resistor_SMD:R_0603_1608Metric, F.Cu at (82.5, 87.2)
- added R35: 10K, Resistor_SMD:R_0603_1608Metric, F.Cu at (86.5, 69.7)
- added R36: 10K, Resistor_SMD:R_0603_1608Metric, F.Cu at (86.5, 72.2)
- added R37: 10K, Resistor_SMD:R_0603_1608Metric, F.Cu at (86.5, 74.7)
- added R38: 10K, Resistor_SMD:R_0603_1608Metric, F.Cu at (86.5, 77.2)
- added R39: 10K, Resistor_SMD:R_0603_1608Metric, F.Cu at (86.5, 79.7)
- added R40: 10K, Resistor_SMD:R_0603_1608Metric, F.Cu at (86.5, 82.2)
- added R41: 10K, Resistor_SMD:R_0603_1608Metric, F.Cu at (86.5, 84.7)
- added R42: 10K, Resistor_SMD:R_0603_1608Metric, F.Cu at (86.5, 87.2)
- added R43: 10K, Resistor_SMD:R_0603_1608Metric, F.Cu at (90.5, 69.7)
- added R44: 10K, Resistor_SMD:R_0603_1608Metric, F.Cu at (90.5, 72.2)
- added R45: 10K, Resistor_SMD:R_0603_1608Metric, F.Cu at (90.5, 74.7)
- added R46: 10K, Resistor_SMD:R_0603_1608Metric, F.Cu at (90.5, 77.2)
- added R47: 10K, Resistor_SMD:R_0603_1608Metric, F.Cu at (90.5, 79.7)
- added R48: 10K, Resistor_SMD:R_0603_1608Metric, F.Cu at (90.5, 82.2)
- added R49: 10K, Resistor_SMD:R_0603_1608Metric, F.Cu at (90.5, 84.7)
- added R50: 10K, Resistor_SMD:R_0603_1608Metric, F.Cu at (90.5, 87.2)
- added R51: 1M, Resistor_SMD:R_0603_1608Metric, F.Cu at (194.1, 67.5)
- added R63: 1M, Resistor_SMD:R_0603_1608Metric, F.Cu at (201.4, 40.8)
- added R75: 4.7k, Resistor_SMD:R_0603_1608Metric, F.Cu at (232.2, 80.0)
- added R76: 4.7k, Resistor_SMD:R_0603_1608Metric, F.Cu at (232.2, 82.5)
- added R77: 4.7k, Resistor_SMD:R_0603_1608Metric, F.Cu at (232.2, 85.0)
- added R78: 4.7k, Resistor_SMD:R_0603_1608Metric, F.Cu at (232.2, 87.5)
- added R79: 1M, Resistor_SMD:R_0603_1608Metric, F.Cu at (232.2, 90.0)
- added R80: 90.9kΩ ±1%, Resistor_SMD:R_0603_1608Metric, F.Cu at (236.2, 62.4)
- added R81: 10kΩ ±1%, Resistor_SMD:R_0603_1608Metric, F.Cu at (236.2, 64.9)
- added R82: 5.1k, Resistor_SMD:R_0603_1608Metric, F.Cu at (236.2, 67.4)
- added R83: 5.1k, Resistor_SMD:R_0603_1608Metric, F.Cu at (236.2, 69.9)
- added R84: 1M, Resistor_SMD:R_0603_1608Metric, F.Cu at (236.2, 72.5)
- added R85: 9.53kΩ ±1%, Resistor_SMD:R_0603_1608Metric, F.Cu at (236.2, 75.0)
- added R86: 10k, Resistor_SMD:R_0603_1608Metric, F.Cu at (223.4, 110.1)
- added R87: 4.7k, Resistor_SMD:R_0603_1608Metric, F.Cu at (236.2, 80.0)
- added R88: 4.7k, Resistor_SMD:R_0603_1608Metric, F.Cu at (236.2, 82.5)
- added R89: 4.7k, Resistor_SMD:R_0603_1608Metric, F.Cu at (236.2, 85.0)
- added R90: 1M, Resistor_SMD:R_0603_1608Metric, F.Cu at (236.2, 87.5)
- added R91: 1M, Resistor_SMD:R_0603_1608Metric, F.Cu at (236.2, 90.0)
- added R92: 5.1k, Resistor_SMD:R_0603_1608Metric, F.Cu at (240.2, 62.4)
- added R93: 5.1k, Resistor_SMD:R_0603_1608Metric, F.Cu at (240.2, 64.9)
- added R94: 10k, Resistor_SMD:R_0603_1608Metric, F.Cu at (240.2, 67.4)
- added R95: 10k, Resistor_SMD:R_0603_1608Metric, F.Cu at (240.2, 69.9)
- added R96: 25.5k, Resistor_SMD:R_0603_1608Metric, F.Cu at (240.2, 72.5)
- added R97: 1M, Resistor_SMD:R_0603_1608Metric, F.Cu at (240.2, 75.0)
- added R98: 5.1k, Resistor_SMD:R_0603_1608Metric, F.Cu at (240.2, 77.5)
- added R99: 10k, Resistor_SMD:R_0603_1608Metric, F.Cu at (240.2, 80.0)
- added RE2: EC11, Rotary_Encoder:RotaryEncoder_Alps_EC11E-Switch_Vertical_H20mm, F.Cu at (137.8, -7.28)
- added RE3: EC11, Rotary_Encoder:RotaryEncoder_Alps_EC11E-Switch_Vertical_H20mm, F.Cu at (137.8, 7.97)
- added RE4: EC11, Rotary_Encoder:RotaryEncoder_Alps_EC11E-Switch_Vertical_H20mm, F.Cu at (137.8, 23.2)
- added RE5: EC11, Rotary_Encoder:RotaryEncoder_Alps_EC11E-Switch_Vertical_H20mm, F.Cu at (137.8, 38.5)
- added RGB1: WS2812B, LED_SMD:LED_WS2812B_PLCC4_5.0x5.0mm_P3.2mm, F.Cu at (140.0, -153.1)
- added RGB10: WS2812B, LED_SMD:LED_WS2812B_PLCC4_5.0x5.0mm_P3.2mm, F.Cu at (148.4, -133.3)
- added RGB100: WS2812B, LED_SMD:LED_WS2812B_PLCC4_5.0x5.0mm_P3.2mm, F.Cu at (64.2, 71.7)
- added RGB101: WS2812B, LED_SMD:LED_WS2812B_PLCC4_5.0x5.0mm_P3.2mm, F.Cu at (64.2, 78.3)
- added RGB102: WS2812B, LED_SMD:LED_WS2812B_PLCC4_5.0x5.0mm_P3.2mm, F.Cu at (64.2, 85.0)
- added RGB103: WS2812B, LED_SMD:LED_WS2812B_PLCC4_5.0x5.0mm_P3.2mm, F.Cu at (64.2, 91.6)
- added RGB104: WS2812B, LED_SMD:LED_WS2812B_PLCC4_5.0x5.0mm_P3.2mm, F.Cu at (64.2, 98.2)
- added RGB11: WS2812B, LED_SMD:LED_WS2812B_PLCC4_5.0x5.0mm_P3.2mm, F.Cu at (148.4, -126.7)
- added RGB12: WS2812B, LED_SMD:LED_WS2812B_PLCC4_5.0x5.0mm_P3.2mm, F.Cu at (148.4, -120.0)
- added RGB13: WS2812B, LED_SMD:LED_WS2812B_PLCC4_5.0x5.0mm_P3.2mm, F.Cu at (156.8, -153.1)
- added RGB14: WS2812B, LED_SMD:LED_WS2812B_PLCC4_5.0x5.0mm_P3.2mm, F.Cu at (156.8, -146.5)
- added RGB15: WS2812B, LED_SMD:LED_WS2812B_PLCC4_5.0x5.0mm_P3.2mm, F.Cu at (156.8, -139.9)
- added RGB16: WS2812B, LED_SMD:LED_WS2812B_PLCC4_5.0x5.0mm_P3.2mm, F.Cu at (156.8, -133.3)
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Routing:
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Other:
- board size 181 x 114.3 mm -> 181 x 150 mm
- copper layers 2 -> 4

Commit message: started hub design
Parts:
- R80, R81, R83: moved to B.Cu
- moved R80 49.3 mm to (216.8, 107.7)
- moved R81 48.4 mm to (216.8, 109.2), turned to 180 degrees
- moved C197 42.0 mm to (245.6, 111.0)
- moved R83 38.3 mm to (215.6, 102.2)
- moved R85 35.6 mm to (239.6, 110.4)
- moved U17 33.7 mm to (224.5, 109.6)
- moved C198 32.9 mm to (245.6, 112.9)
- moved C184 28.4 mm to (231.1, 112.5), turned to -90 degrees
- moved R87 27.7 mm to (224.4, 105.1), turned to 180 degrees
- moved R89 24.6 mm to (224.4, 106.6), turned to 180 degrees
- moved R88 24.1 mm to (224.4, 103.6), turned to 180 degrees
- moved U20 22.1 mm to (224.9, 97.7), turned to 90 degrees
- moved C173 11.4 mm to (224.2, 100.7), turned to 180 degrees
- moved C185 11.0 mm to (229.7, 97.0), turned to 90 degrees
- moved C186 7.98 mm to (228.0, 97.0), turned to 90 degrees
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Routing:
- net /USB Hub/1V1_HUB: track 0.00 -> 9.36 mm
- net /USB Hub/BAT_EN_4: track 0.00 -> 5.74 mm
- net GND: track 1409.2 -> 1414.3 mm
- net /USB Hub/~{OVCURR2}: track 0.00 -> 4.99 mm
- net /USB Hub/BAT_EN_3: track 0.00 -> 3.91 mm
- net Net-(U16-USB_R1): track 0.00 -> 3.71 mm
- net Net-(U16-TEST): track 0.00 -> 3.50 mm
- net +3V3: track 0.00 -> 3.47 mm
- net Net-(U16-GANGED/SMBA2/HS_UP): track 0.00 -> 3.44 mm
- net Net-(U16-FULLPWRMGMTz/SMBA1/SS_UP): track 0.00 -> 3.36 mm
- net /USB Hub/~{OVCURR1}: track 0.00 -> 3.32 mm
- net Net-(U16-GRSTz): track 0.00 -> 3.21 mm
- net Net-(U16-AUTOENz/HS_SUSPEND): track 0.00 -> 3.14 mm
- net +5V: track 1485.3 -> 1486.1 mm
- net /USB Hub/UP_VBUS: track 0.00 -> 0.50 mm
