File: Schematics and PCB/Schematics and PCB.kicad_sch (KiCad schematic)
At the start: 3 parts, among them J1 Magnetic Left, J2 Magnetic Right, U1 SN74AUC1G126DBVR

Commit message: minor changes
Parts:
- removed J1: Magnetic Left, symbol Connector_Generic:Conn_01x05
- removed J2: Magnetic Right, symbol Connector_Generic:Conn_01x05
- removed U1: SN74AUC1G126DBVR, symbol mechpadLibrary:Tri-state_Buffer
Connections:
- no-connect marks 1 -> 0
Other:
- removed sheet Main IC
- removed sheet Main IC1
- removed sheet Main IC2
- removed sheet Shift Register
- removed sheet Shift Register1
- removed sheet Shift Register2
- added sheet Microcontroller (microcontroller.kicad_sch)
- sheet Left Switch Matrix ports: added COL0, COL1, COL2, COL3, COL4, COL5, COL6, RGB_IN, RGB_OUT, ROW0, ROW1, ROW2, ROW3, ROW4, ROW5; removed +5V, COL_0_L, COL_1_L, COL_2_L, COL_3_L, COL_4_L, COL_5_L, COL_6_L, GND, RGB_IN_L, RGB_OUT_L, ROW_0_L, ROW_1_L, ROW_2_L, ROW_3_L, ROW_4_L, ROW_5_L
- sheet Li-Po Charge Boost ports: added 5V_USB; removed +1V1, +3V3, 1V1_EN, 3V3_EN, 5V_BAT, 5V_IN, GND
- sheet Numpad Switch Matrix ports: added COL0, COL1, COL2, COL3, RE_A_0, RE_A_1, RE_A_2, RE_A_3, RE_B_0, RE_B_1, RE_B_2, RE_B_3, RGB_IN, RGB_OUT, ROW0, ROW1, ROW2, ROW3, ROW4, ROW5; removed +5V, COL_0_N, COL_1_N, COL_2_N, COL_3_N, GND, RE_1_A, RE_1_B, RE_2_A, RE_2_B, RE_3_A, RE_3_B, RE_4_A, RE_4_B, RGB_IN_N, RGB_OUT_N, ROW_0_N, ROW_1_N, ROW_2_N, ROW_3_N, ROW_4_N, ROW_5_N
- sheet Right Switch Matrix ports: added COL0, COL1, COL2, COL3, COL4, COL5, COL6, COL7, COL8, RE_A, RE_B, RGB_IN, RGB_OUT, ROW0, ROW1, ROW2, ROW3, ROW4, ROW5; removed +5V, COL_0_R, COL_1_R, COL_2_R, COL_3_R, COL_4_R, COL_5_R, COL_6_R, COL_7_R, COL_8_R, GND, RE_1_A, RE_1_B, RGB_IN_R, RGB_OUT_R, ROW_0_R, ROW_1_R, ROW_2_R, ROW_3_R, ROW_4_R, ROW_5_R
- sheet USB Hub ports: added DN4_VCC; removed +1V1, +3V3, +5V, GND
