File: Schematics and PCB/Schematics and PCB.kicad_sch (KiCad schematic)
At the start: 0 parts

Commit message: layout improvements
Parts:
- added R1, R2, R3: 10k, Resistor_SMD:R_0603_1608Metric, symbol Device:R_US
Connections:
- new net GND: R1.2, R2.2, R3.2
- new net Magnetic connectors L/RGB DETECT: R1.1
- new net Magnetic connectors N/RGB DETECT: R3.1
- new net Magnetic connectors R/RGB DETECT: R2.1
- no-connect marks 0 -> 34
Other:
- sheet Li-Po Charge Boost renamed Li-Po Charge Boost R
- sheet Microcontroller renamed Microcontroller R
- sheet USB Hub renamed USB Hub R
- added sheet Li-Po Charge Boost L (Li-Po_Charge_Boost.kicad_sch)
- added sheet Li-Po Charge Boost N (Li-Po_Charge_Boost.kicad_sch)
- added sheet Magnetic connectors L (magneticConnectors.kicad_sch)
- added sheet Magnetic connectors N (magneticConnectors.kicad_sch)
- added sheet Magnetic connectors R (magneticConnectors.kicad_sch)
- added sheet Microcontroller L (microcontroller.kicad_sch)
- added sheet Microcontroller N (microcontroller.kicad_sch)
- added sheet USB Hub L (USB_Hub.kicad_sch)
- added sheet USB Hub N (USB_Hub.kicad_sch)
- sheet Microcontroller R ports: added GPIO1, GPIO10, GPIO11, GPIO12, GPIO13, GPIO14, GPIO15, GPIO16, GPIO17, GPIO18, GPIO2, GPIO21, GPIO3, GPIO38, GPIO39, GPIO4, GPIO40, GPIO41, GPIO42, GPIO43, GPIO44, GPIO45, GPIO46, GPIO47, GPIO48, GPIO5, GPIO6, GPIO7, GPIO8, GPIO9, USB_N, USB_P; removed D+, D-
- note added: "Left board"
- note added: "Numpad"
- note added: "Right board"
