File: Schematics and PCB/USB_Hub.kicad_sch (KiCad schematic)
At the start: 95 parts, among them J3 DOWNSTREAM_1, J4 DOWNSTREAM_1, J6 UPSTREAM, J8 DOWNSTREAM_1, U17 TUSB8042A, U18 TPS2561, U19 TPS2561, Y1 24MHz

Commit message: layout improvements
Parts:
- removed D120: DESD5V0U1BA, Diode_SMD:D_SOD-323_HandSoldering, symbol Device:D_TVS
- added C288, C303, C307, C308: 100n, Capacitor_SMD:C_0603_1608Metric, symbol Device:C
- added C291: 33p, Capacitor_SMD:C_0603_1608Metric, symbol Device:C
- added C294, C310: 22u, Capacitor_SMD:C_Elec_4x5.4, symbol Device:C_Polarized_US
- added C300, C306: 10u, Capacitor_SMD:C_Elec_4x5.4, symbol Device:C_Polarized_US
- added D120, D121, D122, D123, D124: LESD5D5.0CT1G, Diode_SMD:D_SOD-523, symbol Diode:SMAJ5.0CA
- added L4: 3u6, Inductor_SMD:L_0805_2012Metric, symbol Device:L
- added L7: 2u, Inductor_SMD:L_0805_2012Metric, symbol Device:L
- added R157: 115k, Resistor_SMD:R_0603_1608Metric, symbol Device:R_US
- added R160: 25.5k, Resistor_SMD:R_0603_1608Metric, symbol Device:R_US
- added R163, R164: 10k, Resistor_SMD:R_0603_1608Metric, symbol Device:R_US
- added U28, U31: RT7295A, Package_TO_SOT_SMD:TSOT-23-6, symbol mechpadLibrary:RT7295A
- C131: renamed from C4; footprint (none) -> Capacitor_SMD:C_0603_1608Metric
- C132: renamed from C3; footprint (none) -> Capacitor_SMD:C_0603_1608Metric
- C133: renamed from C162; footprint (none) -> Capacitor_SMD:C_Elec_4x5.4
- C134: renamed from C163; footprint Capacitor_SMD:C_0201_0603Metric -> Capacitor_SMD:C_0603_1608Metric
- C135: renamed from C164; footprint Capacitor_SMD:C_0201_0603Metric -> Capacitor_SMD:C_0603_1608Metric
- C136: renamed from C172; footprint (none) -> Capacitor_SMD:C_0603_1608Metric
- C137: renamed from C173; footprint (none) -> Capacitor_SMD:C_0603_1608Metric
- C138: renamed from C174; footprint (none) -> Capacitor_SMD:C_0603_1608Metric
- C139: renamed from C175; footprint (none) -> Capacitor_SMD:C_0603_1608Metric
- C140: renamed from C176; footprint (none) -> Capacitor_SMD:C_Elec_4x5.4
- C141: renamed from C5; footprint (none) -> Capacitor_SMD:C_0603_1608Metric
- C142: renamed from C6; footprint (none) -> Capacitor_SMD:C_0603_1608Metric
- C143: renamed from C10; footprint (none) -> Capacitor_SMD:C_0603_1608Metric
- C144: renamed from C182; footprint (none) -> Capacitor_SMD:C_0603_1608Metric
- C145: renamed from C183; footprint (none) -> Capacitor_SMD:C_0603_1608Metric
- C146: renamed from C184; footprint (none) -> Capacitor_SMD:C_0603_1608Metric
- C147: renamed from C185; footprint (none) -> Capacitor_SMD:C_0603_1608Metric
- C148: renamed from C186; footprint (none) -> Capacitor_SMD:C_0603_1608Metric
- C149: renamed from C187; footprint (none) -> Capacitor_SMD:C_0603_1608Metric
- C150: renamed from C188; footprint (none) -> Capacitor_SMD:C_0603_1608Metric
- C151: renamed from C189; footprint (none) -> Capacitor_SMD:C_Elec_4x5.4
- C152: renamed from C8; footprint Capacitor_SMD:C_0201_0603Metric -> Capacitor_SMD:C_0603_1608Metric
- C153: renamed from C9; footprint Capacitor_SMD:C_0201_0603Metric -> Capacitor_SMD:C_0603_1608Metric
- C154: renamed from C7; footprint (none) -> Capacitor_SMD:C_0603_1608Metric
- C155: renamed from C11; footprint (none) -> Capacitor_SMD:C_0603_1608Metric
- C156: renamed from C12; footprint (none) -> Capacitor_SMD:C_0603_1608Metric
- C157: renamed from C1; footprint (none) -> Capacitor_SMD:C_0603_1608Metric
- C158: renamed from C2; footprint (none) -> Capacitor_SMD:C_0603_1608Metric
- C159: renamed from C13; footprint Capacitor_SMD:C_0201_0603Metric -> Capacitor_SMD:C_0603_1608Metric
- C160: renamed from C14; footprint Capacitor_SMD:C_0201_0603Metric -> Capacitor_SMD:C_0603_1608Metric
- C161: renamed from C167; footprint (none) -> Capacitor_SMD:C_0603_1608Metric
- C162: renamed from C15; footprint (none) -> Capacitor_SMD:C_0603_1608Metric
- C163: renamed from C101; footprint (none) -> Capacitor_SMD:C_0603_1608Metric
- C164: renamed from C130; footprint (none) -> Capacitor_SMD:C_0603_1608Metric
- C165: renamed from C193; footprint (none) -> Capacitor_SMD:C_0603_1608Metric
- C166: renamed from C195; footprint (none) -> Capacitor_SMD:C_0603_1608Metric
- C167: renamed from C196; footprint (none) -> Capacitor_SMD:C_0603_1608Metric
- C168: renamed from C197; footprint (none) -> Capacitor_SMD:C_0603_1608Metric
- C169: renamed from C198; footprint (none) -> Capacitor_SMD:C_0603_1608Metric
- C170: renamed from C131; footprint Capacitor_SMD:C_0201_0603Metric -> Capacitor_SMD:C_0603_1608Metric
- C171: renamed from C132; footprint Capacitor_SMD:C_0201_0603Metric -> Capacitor_SMD:C_0603_1608Metric
- C172: renamed from C133; footprint (none) -> Capacitor_SMD:C_0603_1608Metric
- C173: renamed from C203; footprint (none) -> Capacitor_SMD:C_0603_1608Metric
- C174: renamed from C204; footprint (none) -> Capacitor_SMD:C_0603_1608Metric
- C175: renamed from C205; footprint (none) -> Capacitor_SMD:C_0603_1608Metric
- C176: renamed from C206; footprint (none) -> Capacitor_SMD:C_0603_1608Metric
- C177: renamed from C134; footprint (none) -> Capacitor_SMD:C_0603_1608Metric
- FB1: renamed from FB7; footprint (none) -> Inductor_SMD:L_0603_1608Metric
- FB2: renamed from FB1; footprint (none) -> Inductor_SMD:L_0603_1608Metric
- FB3: renamed from FB10; footprint (none) -> Inductor_SMD:L_0603_1608Metric
- FB4: renamed from FB2; footprint (none) -> Inductor_SMD:L_0603_1608Metric
- FB5: renamed from FB3; footprint (none) -> Inductor_SMD:L_0603_1608Metric
- FB6: renamed from FB4; footprint (none) -> Inductor_SMD:L_0603_1608Metric
- J1: renamed from J6; footprint (none) -> Connector_USB:USB_C_Receptacle_Molex_105450-0101
- J2: renamed from J8; footprint (none) -> Connector_USB:USB_C_Receptacle_Molex_105450-0101
- J3, J4: footprint (none) -> Connector_USB:USB_C_Receptacle_Molex_105450-0101
- R47: renamed from R2; footprint Resistor_SMD:R_0402_1005Metric -> Resistor_SMD:R_0603_1608Metric
- R48: renamed from R3; footprint Resistor_SMD:R_0402_1005Metric -> Resistor_SMD:R_0603_1608Metric
- R49: renamed from R5; footprint (none) -> Resistor_SMD:R_0603_1608Metric
- R50: renamed from R6; footprint (none) -> Resistor_SMD:R_0603_1608Metric
- R52: renamed from R10; footprint (none) -> Resistor_SMD:R_0603_1608Metric
- R53: renamed from R11; footprint (none) -> Resistor_SMD:R_0603_1608Metric
- R54: renamed from R83; footprint (none) -> Resistor_SMD:R_0603_1608Metric
- R55: renamed from R82; footprint (none) -> Resistor_SMD:R_0603_1608Metric
- R56: renamed from R81; footprint (none) -> Resistor_SMD:R_0603_1608Metric
- R57: renamed from R80; footprint (none) -> Resistor_SMD:R_0603_1608Metric
- R60: renamed from R9; footprint (none) -> Resistor_SMD:R_0603_1608Metric
- R61: renamed from R12; footprint (none) -> Resistor_SMD:R_0603_1608Metric
- R62: renamed from R87; footprint (none) -> Resistor_SMD:R_0603_1608Metric
- R63: renamed from R1; footprint (none) -> Resistor_SMD:R_0603_1608Metric
- R64: renamed from R88; footprint (none) -> Resistor_SMD:R_0603_1608Metric
- R65: renamed from R89; footprint (none) -> Resistor_SMD:R_0603_1608Metric
- R66: renamed from R90; footprint (none) -> Resistor_SMD:R_0603_1608Metric
- R67: renamed from R91; footprint (none) -> Resistor_SMD:R_0603_1608Metric
- R69: renamed from R96; footprint (none) -> Resistor_SMD:R_0603_1608Metric
- R70: renamed from R97; footprint (none) -> Resistor_SMD:R_0603_1608Metric
- R71: renamed from R32; footprint (none) -> Resistor_SMD:R_0603_1608Metric
- R72: renamed from R53; footprint (none) -> Resistor_SMD:R_0603_1608Metric
- R73: renamed from R98; footprint (none) -> Resistor_SMD:R_0603_1608Metric
- R74: renamed from R101; footprint (none) -> Resistor_SMD:R_0603_1608Metric
- R75: renamed from R102; footprint (none) -> Resistor_SMD:R_0603_1608Metric
- R76: renamed from R104; footprint (none) -> Resistor_SMD:R_0603_1608Metric
- U8: renamed from U17; footprint (none) -> Package_DFN_QFN:VQFN-64-1EP_9x9mm_P0.5mm_EP5.4x5.4mm_ThermalVias
- Y1: footprint (none) -> Crystal:Crystal_SMD_3225-4Pin_3.2x2.5mm
- renumbered D121 to D119, F2 to F1, R4 to R46, R7 to R51, R8 to R58, R86 to R59, R31 to R68, U19 to U10, U18 to U9
Connections:
- net +1V1: now also C310.1, L7.2, R163.1
- net +3V3: now also C291.1, C294.1, L4.2, R157.1
- net 5V fused: now also D120.2 (A2)
- net DN1_VBUS: now also D121.2 (A2)
- net DN2_VBUS: now also D122.2 (A2)
- net DN3_VBUS: now also D123.2 (A2)
- net DN4_VBUS: now also D124.2 (A2)
- net GND: now also C294.2, C300.2, C303.2, C306.2, C307.2, C310.2, D120.1 (A1), D121.1 (A1), D122.1 (A1), D123.1 (A1), D124.1 (A1), R160.2, R164.2, U28.2 (GND), U31.2 (GND)
- net UP_VBUS renamed +5V
- net +5V: now also C300.1, C303.1, C306.1, C307.1, U28.4 (EN), U28.5 (VCC), U31.4 (EN), U31.5 (VCC)
- new net: C288.1, U28.1 (BOOT)
- new net: C288.2, L4.1, U28.6 (SW)
- new net: C291.2, R157.2, R160.1, U28.3 (FB)
- new net: C308.1, U31.1 (BOOT)
- new net: R163.2, R164.1, U31.3 (FB)
- new net: C308.2, L7.1, U31.6 (SW)
Other:
- note added: "1.1V regulator"
- note added: "3.3V regulator"
- moved on the sheet: C131, C132, C133, C134, C135, C136, C137, C138, C139, C140, C141, C142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
