File: Schematics and PCB/microcontroller.kicad_sch (KiCad schematic)
At the start: 34 parts, among them J2 USB C 2.0, Q2 L8050QLT1G, Q3 L8050QLT1G, U4 ESP32-S3-WROOM-2, U5 CP2102N-Axx-xQFN28

Commit message: layout improvements
Parts:
- removed C18, C21, C22: 100n, symbol Device:C
- removed C19: 1n, symbol Device:C
- removed C20, C23: 10u, symbol Device:C_Polarized_US
- removed C24: 1u, symbol Device:C
- removed D2: 1N5819HW-7-F, Diode_SMD:D_SOD-123, symbol Device:D
- removed D3, D4, D5: LESD5D5.0CT1G, Diode_SMD:D_SOD-523, symbol Diode:SMAJ5.0CA
- removed FB5: >50mΩ 220Ω @ 100MHz, symbol Device:FerriteBead
- removed J2: USB C 2.0, symbol mechpadLibrary:USB_C_Receptacle_2.0
- removed Q2, Q3: L8050QLT1G, symbol Simulation_SPICE:NPN
- removed R33: 1M, Resistor_SMD:R_0603_1608Metric, symbol Device:R_US
- removed R34, R35: 5.1k, symbol Device:R_US
- removed R36, R37, R40, R41, R42: 10k, symbol Device:R_US
- removed R38: 22k1 (1%), symbol Device:R_US
- removed R39: 47k5 (1%), symbol Device:R_US
- removed U5: CP2102N-Axx-xQFN28, Package_DFN_QFN:QFN-28-1EP_5x5mm_P0.5mm_EP3.35x3.35mm, symbol Interface_USB:CP2102N-Axx-xQFN28
- added C297: 1u, Capacitor_SMD:C_0603_1608Metric, symbol Device:C
- added C309, C317: 100n, Capacitor_SMD:C_0603_1608Metric, symbol Device:C
- added R169, R172: 10k, Resistor_SMD:R_0603_1608Metric, symbol Device:R_US
- added SW105: BOOT, ESC-TFG-KiCad:SPDT, symbol Switch:SW_SPST
- added SW108: RESET, ESC-TFG-KiCad:SPDT, symbol Switch:SW_SPST
- C127: renamed from C16; footprint (none) -> Capacitor_SMD:C_0603_1608Metric
- C128: renamed from C17; footprint (none) -> Capacitor_SMD:C_Elec_4x5.4
- R42: renamed from R30; footprint (none) -> Resistor_SMD:R_0603_1608Metric
- R43: renamed from R29; footprint (none) -> Resistor_SMD:R_0603_1608Metric
- renumbered D1 to D113, D6 to D114, D116 to D115, U4 to U6
Connections:
- net +3V3: now also R169.2, R172.2; no longer U6.3 (EN)
- net GND: now also C297.2, C309.2, C317.2, SW105.1 (A), SW108.2 (B)
- net GPIO17: now reaches U6.10 (IO17)
- net GPIO18: now reaches U6.11 (IO18)
- net GPIO8: now reaches U6.12 (IO8)
- net GPIO3: now reaches U6.15 (IO3)
- net GPIO46: now reaches U6.16 (IO46)
- net GPIO9: now reaches U6.17 (IO9)
- net GPIO10: now reaches U6.18 (IO10)
- net GPIO11: now reaches U6.19 (IO11)
- net GPIO12: now reaches U6.20 (IO12)
- net GPIO13: now reaches U6.21 (IO13)
- net GPIO14: now reaches U6.22 (IO14)
- net GPIO21: now reaches U6.23 (IO21)
- net GPIO47: now reaches U6.24 (IO47)
- net GPIO48: now reaches U6.25 (IO48)
- net GPIO45: now reaches U6.26 (IO45)
- net at U6.27 (IO0): now also C309.1, R172.1, SW105.2 (B)
- net GPIO38: now reaches U6.31 (IO38)
- net GPIO39: now reaches U6.32 (MTCK/IO39)
- net GPIO40: now reaches U6.33 (MTDO/IO40)
- net GPIO41: now reaches U6.34 (MTDI/IO41)
- net GPIO42: now reaches U6.35 (MTMS/IO42)
- net GPIO44: now reaches U6.36 (RXD0/IO44)
- net GPIO43: now reaches U6.37 (TXD0/IO43)
- net GPIO2: now reaches U6.38 (IO2)
- net GPIO1: now reaches U6.39 (IO1)
- net GPIO4: now reaches U6.4 (IO4)
- net GPIO5: now reaches U6.5 (IO5)
- net GPIO6: now reaches U6.6 (IO6)
- net GPIO7: now reaches U6.7 (IO7)
- net GPIO15: now reaches U6.8 (IO15)
- net GPIO16: now reaches U6.9 (IO16)
- new net: C297.1, C317.1, R169.1, SW108.1 (A), U6.3 (EN)
- no-connect marks 17 -> 0
Other:
- note removed: "Programming USB C port"
- moved on the sheet: D114, D115, R42, R43, U6
